Commit message: 1 mecanum wheel attached with proper TFs and joints in gazebo

File: linorobot2_description/urdf/mech/mecanum_wheel_left.urdf.xacro (robot description, xacro)
@@ -16,5 +16,5 @@
           iyz="-1.66085499471637E-18"
           izz="3.76577202480009E-05" />
-    </inertial>
+      </inertial>
       <visual>
         <origin
@@ -46,5 +46,5 @@
       <child link="${end}_${side}_wheel" />
       <axis xyz="0 1 0" />
-      <dynamics damping="0.1" friction="0.01"/>
+      <!--<dynamics damping="0.1" friction="0.01"/>-->
     </joint>
     <link
@@ -63,5 +63,5 @@
           iyz="4.06169630282727E-21"
           izz="8.39719993847474E-05" />
-    </inertial>
+      </inertial>
       <visual>
         <origin
@@ -116,5 +116,5 @@
           iyz="2.75305456980319E-21"
           izz="8.39719993847476E-05" />
-    </inertial>
+      </inertial>
       <visual>
         <origin
@@ -169,5 +169,5 @@
           iyz="-8.0163727523739E-19"
           izz="3.31951561004127E-07" />
-    </inertial>
+      </inertial>
       <visual>
         <origin
@@ -206,5 +206,5 @@
       <axis
         xyz="0 0 1" />
-      <dynamics damping="0.1" friction="0.01"/>
+      <!--<dynamics damping="0.1" friction="0.01"/>-->
     </joint>
     <link
@@ -223,5 +223,5 @@
           iyz="-8.0163727523739E-19"
           izz="3.31951561004127E-07" />
-    </inertial>
+     </inertial>
       <visual>
         <origin
@@ -260,5 +260,5 @@
       <axis
         xyz="0 0 1" />
-      <dynamics damping="0.1" friction="0.01"/>
+      <!--<dynamics damping="0.1" friction="0.01"/>-->
     </joint>
     <link
@@ -314,5 +314,5 @@
       <axis
         xyz="0 0 1" />
-      <dynamics damping="0.1" friction="0.01"/>
+      <!--<dynamics damping="0.1" friction="0.01"/>-->
     </joint>
     <link
@@ -368,5 +368,5 @@
       <axis
         xyz="0 0 1" />
-      <dynamics damping="0.1" friction="0.01"/>
+      <!--<dynamics damping="0.1" friction="0.01"/>-->
     </joint>
     <link
@@ -422,5 +422,5 @@
       <axis
         xyz="0 0 1" />
-      <dynamics damping="0.1" friction="0.01"/>
+      <!--<dynamics damping="0.1" friction="0.01"/>-->
     </joint>
     <link
@@ -476,5 +476,5 @@
       <axis
         xyz="0 0 1" />
-      <dynamics damping="0.1" friction="0.01"/>
+      <!--<dynamics damping="0.1" friction="0.01"/>-->
     </joint>
     <link
@@ -530,5 +530,5 @@
       <axis
         xyz="0 0 1" />
-      <dynamics damping="0.1" friction="0.01"/>
+      <!--<dynamics damping="0.1" friction="0.01"/>-->
     </joint>
     <link
@@ -584,5 +584,5 @@
       <axis
         xyz="0 0 1" />
-      <dynamics damping="0.1" friction="0.01"/>
+      <!--<dynamics damping="0.1" friction="0.01"/>-->
     </joint>
     <link
@@ -638,5 +638,5 @@
       <axis
         xyz="0 0 1" />
-      <dynamics damping="0.1" friction="0.01"/>
+      <!--<dynamics damping="0.1" friction="0.01"/>-->
     </joint>
     <link
@@ -692,5 +692,5 @@
       <axis
         xyz="0 0 1" />
-      <dynamics damping="0.1" friction="0.01"/>
+      <!--<dynamics damping="0.1" friction="0.01"/>-->
     </joint>
     <link
@@ -746,5 +746,5 @@
       <axis
         xyz="0 0 1" />
-      <dynamics damping="0.1" friction="0.01"/>
+      <!--<dynamics damping="0.1" friction="0.01"/>-->
     </joint>
     <link
@@ -800,5 +800,5 @@
       <axis
         xyz="0 0 1" />
-      <dynamics damping="0.1" friction="0.01"/>
+      <!--<dynamics damping="0.1" friction="0.01"/>-->
     </joint>
     <link
@@ -854,5 +854,5 @@
       <axis
         xyz="0 0 1" />
-      <dynamics damping="0.1" friction="0.01"/>
+      <!--<dynamics damping="0.1" friction="0.01"/>-->
     </joint>
     <link
@@ -908,5 +908,5 @@
       <axis
         xyz="0 0 1" />
-      <dynamics damping="0.1" friction="0.01"/>
+      <!--<dynamics damping="0.1" friction="0.01"/>-->
     </joint>
     <link
@@ -962,5 +962,5 @@
       <axis
         xyz="0 0 1" />
-      <dynamics damping="0.1" friction="0.01"/>
+      <!--<dynamics damping="0.1" friction="0.01"/>-->
     </joint>
   </xacro:macro>

File: linorobot2_description/urdf/robots/mecanum.urdf.xacro (robot description, xacro)
@@ -45,5 +45,5 @@
     mass="${wheel_mass}"
   />
-  <xacro:mecanum_wheel_right
+  <!-- <xacro:mecanum_wheel_right
     side="right"
     end="front"
@@ -54,7 +54,7 @@
     pos_z="${wheel_pos_z}"
     mass="${wheel_mass}"
-  />
+  /> -->
   <!-- Back wheels mechanum style swapped (left mecanum wheel goes on right side of robot, and vice versa) -->
-  <xacro:mecanum_wheel_right
+  <!-- <xacro:mecanum_wheel_right
     side="left"
     end="rear"
@@ -75,5 +75,5 @@
     pos_z="${wheel_pos_z}"
     mass="${wheel_mass}"
-  />
+  /> -->
   <!-- IsaacSim will likely not respect joint angles for realsense joints -->
   <joint
