Commit message: All 4 cameras on drone properly attached to drone and spitting out colour, depth, and pointclouds. Cleaned up camera urdf xacro

File: linorobot2_description/urdf/mech/side_channel.urdf.xacro (robot description, xacro)
@@ -1,4 +1,4 @@
 <?xml version="1.0"?>
-<robot xmlns:xacro="http://ros.org/wiki/xacro">
+<robot name="linorobot2_mecanum" xmlns:xacro="http://ros.org/wiki/xacro">
   <xacro:macro name="side_channel" params="side pos_y">
     <link name="${side}_channel">

File: linorobot2_description/urdf/robots/mecanum_libplanar.urdf.xacro (robot description, xacro)
@@ -11,4 +11,13 @@
   <xacro:include filename="$(find linorobot2_description)/urdf/mech/end_channel.urdf.xacro" />
   <xacro:include filename="$(find linorobot2_description)/urdf/mech/side_channel.urdf.xacro" />
+  <xacro:include filename="$(find linorobot2_description)/urdf/robots/camera.urdf.xacro" />
+  <xacro:camera camera_pos="front" x="0.410335" y="0" z="0.0892"
+                                   r_rs="-1.57" p_rs="0" yaw_rs="-1.57" />
+  <xacro:camera camera_pos="left" x="0.0" y="0.247" z="0.089"
+                                  r_rs="-1.57" p_rs="0.0" yaw_rs="0"/>
+  <xacro:camera camera_pos="rear" x="-0.41" y="0.0" z="0.089"
+                                  r_rs="-1.57" p_rs="0" yaw_rs="1.57" />
+  <xacro:camera camera_pos="right" x="0" y="-0.247" z="0.089"
+                                  r_rs="-1.57" p_rs="0" yaw_rs="3.14"/>
   <gazebo>
     <plugin name="mecanum_wheel_mimic" filename="libgazebo_ros_planar_move.so">
@@ -90,86 +99,3 @@
     mass="${wheel_mass}"
   />
-  <!-- IsaacSim will likely not respect joint angles for realsense joints -->
-  <joint
-    name="base_link_to_front_rs" type="fixed">
-    <origin
-      xyz="0.410335 0 0.0892"
-      rpy="-1.57 1.57 0" />
-    <parent link="base_link" />
-    <child link="front_rs_depth_optical_frame" />
-  </joint>
-  <link name="front_rs_depth_optical_frame">
-  </link>
-  <link name="rear_rs_depth_optical_frame">
-  </link>
-  <!-- IsaacSim will likely not respect joint angles for realsense joints -->
-  <joint
-    name="base_link_to_rear_rs" type="fixed">
-    <origin
-      xyz="-0.41 0 0.089"
-      rpy="-1.57 -1.57 0" />
-    <parent link="base_link" />
-    <child link="rear_rs_depth_optical_frame" />
-  </joint>
-  <link name="left_rs_depth_optical_frame">
-  </link>
-  <!-- IsaacSim will likely not respect joint angles for realsense joints -->
-  <joint
-    name="base_link_to_left_rs" type="fixed">
-    <origin
-      xyz="0 0.247 0.089"
-      rpy="-1.57 0 0" />
-    <parent link="base_link" />
-    <child link="left_rs_depth_optical_frame" />
-  </joint>
-  <link name="right_rs_depth_optical_frame">
-  </link>
-  <!-- IsaacSim will likely not respect joint angles for realsense joints -->
-  <joint
-    name="base_link_to_right_rs" type="fixed">
-    <origin
-      xyz="0 -0.247 0.089"
-      rpy="1.57 0 3.14" />
-    <parent link="base_link" />
-    <child link="right_rs_depth_optical_frame" />
-  </joint>
-  <gazebo reference="right_rs_depth_optical_frame">
-    <sensor type="depth" name="camera1">
-      <update_rate>30.0</update_rate>
-      <depth_camera name="head">
-        <horizontal_fov>2.96</horizontal_fov>
-        <image>
-          <width>480</width>
-          <height>270</height>
-          <format>R8G8B8</format>
-        </image>
-        <clip>
-          <near>0.02</near>
-          <far>3</far>
-        </clip>
-        <noise>
-          <type>gaussian</type>
-          <!-- Noise is sampled independently per pixel on each frame.
-               That pixel's noise value is added to each of its color
-               channels, which at that point lie in the range [0,1]. -->
-          <mean>0.0</mean>
-          <stddev>0.007</stddev>
-        </noise>
-      </depth_camera>
-      <plugin name="camera_controller" filename="libgazebo_ros_camera.so">
-        <alwaysOn>true</alwaysOn>
-        <updateRate>0.0</updateRate>
-        <cameraName>rrbot/camera1</cameraName>
-        <imageTopicName>image_raw</imageTopicName>
-        <cameraInfoTopicName>camera_info</cameraInfoTopicName>
-        <frameName>right_rs_depth_optical_frame</frameName>
-        <hackBaseline>0.07</hackBaseline>
-        <distortionK1>0.0</distortionK1>
-        <distortionK2>0.0</distortionK2>
-        <distortionK3>0.0</distortionK3>
-        <distortionT1>0.0</distortionT1>
-        <distortionT2>0.0</distortionT2>
-      </plugin>
-    </sensor>
-  </gazebo>
 </robot>
