Commit message: Driving robot around with libplanar movement

File: linorobot2_description/urdf/mech/mecanum_wheel_left_fixed.urdf.xacro (robot description, xacro)
@@ -41,10 +41,8 @@
       </collision>
     </link>
-    <joint name="base_link_to_${end}_${side}_wheel" type="continuous">
+    <joint name="base_link_to_${end}_${side}_wheel" type="fixed">
       <origin xyz="${pos_x} ${pos_y} 0"  rpy="0 0 0" />
       <parent link="base_link" />
       <child link="${end}_${side}_wheel" />
-      <axis xyz="0 1 0" />
-      <dynamics friction="0.1"/>
     </joint>
     <link
@@ -196,5 +194,5 @@
     <joint
       name="${end}_${side}_wheel_to_${end}_${side}_roller1"
-      type="continuous">
+      type="fixed">
       <origin
         xyz="-0.064997 -0.01515 0.019737"
@@ -204,7 +202,4 @@
       <child
         link="${end}_${side}_roller1" />
-      <axis
-        xyz="0 0 1" />
-      <dynamics friction="0.1"/>
     </joint>
     <link
@@ -250,5 +245,5 @@
     <joint
       name="${end}_${side}_wheel_to_${end}_${side}_roller2"
-      type="continuous">
+      type="fixed">
       <origin
         xyz="-0.05135 -0.01515 0.044467"
@@ -258,7 +253,4 @@
       <child
         link="${end}_${side}_roller2" />
-      <axis
-        xyz="0 0 1" />
-      <dynamics friction="0.1"/>
     </joint>
     <link
@@ -304,5 +296,5 @@
     <joint
       name="${end}_${side}_wheel_to_${end}_${side}_roller3"
-      type="continuous">
+      type="fixed">
       <origin
         xyz="-0.028824 -0.01515 0.061508"
@@ -312,7 +304,4 @@
       <child
         link="${end}_${side}_roller3" />
-      <axis
-        xyz="0 0 1" />
-      <dynamics friction="0.1"/>
     </joint>
     <link
@@ -358,5 +347,5 @@
     <joint
       name="${end}_${side}_wheel_to_${end}_${side}_roller4"
-      type="continuous">
+      type="fixed">
       <origin
         xyz="-0.0013143 -0.01515 0.067914"
@@ -366,7 +355,4 @@
       <child
         link="${end}_${side}_roller4" />
-      <axis
-        xyz="0 0 1" />
-      <dynamics friction="0.1"/>
     </joint>
     <link
@@ -412,5 +398,5 @@
     <joint
       name="${end}_${side}_wheel_to_${end}_${side}_roller5"
-      type="continuous">
+      type="fixed">
       <origin
         xyz="0.026423 -0.01515 0.062578"
@@ -420,7 +406,4 @@
       <child
         link="${end}_${side}_roller5" />
-      <axis
-        xyz="0 0 1" />
-      <dynamics friction="0.1"/>
     </joint>
     <link
@@ -466,5 +449,5 @@
     <joint
       name="${end}_${side}_wheel_to_${end}_${side}_roller6"
-      type="continuous">
+      type="fixed">
       <origin
         xyz="0.049591 -0.01515 0.04642"
@@ -474,7 +457,4 @@
       <child
         link="${end}_${side}_roller6" />
-      <axis
-        xyz="0 0 1" />
-      <dynamics friction="0.1"/>
     </joint>
     <link
@@ -520,5 +500,5 @@
     <joint
       name="${end}_${side}_wheel_to_${end}_${side}_roller7"
-      type="continuous">
+      type="fixed">
       <origin
         xyz="0.064184 -0.01515 0.022237"
@@ -528,7 +508,4 @@
       <child
         link="${end}_${side}_roller7" />
-      <axis
-        xyz="0 0 1" />
-      <dynamics friction="0.1"/>
     </joint>
     <link
@@ -574,5 +551,5 @@
     <joint
       name="${end}_${side}_wheel_to_${end}_${side}_roller8"
-      type="continuous">
+      type="fixed">
       <origin
         xyz="0.06768 -0.01515 -0.0057919"
@@ -582,7 +559,4 @@
       <child
         link="${end}_${side}_roller8" />
-      <axis
-        xyz="0 0 1" />
-      <dynamics friction="0.1"/>
     </joint>
     <link
@@ -628,5 +602,5 @@
     <joint
       name="${end}_${side}_wheel_to_${end}_${side}_roller9"
-      type="continuous">
+      type="fixed">
       <origin
         xyz="0.059473 -0.01515 -0.032819"
@@ -636,7 +610,4 @@
       <child
         link="${end}_${side}_roller9" />
-      <axis
-        xyz="0 0 1" />
-      <dynamics friction="0.1"/>
     </joint>
     <link
@@ -682,5 +653,5 @@
     <joint
       name="${end}_${side}_wheel_to_${end}_${side}_roller10"
-      type="continuous">
+      type="fixed">
       <origin
         xyz="0.040982 -0.01515 -0.054171"
@@ -690,7 +661,4 @@
       <child
         link="${end}_${side}_roller10" />
-      <axis
-        xyz="0 0 1" />
-      <dynamics friction="0.1"/>
     </joint>
     <link
@@ -736,5 +704,5 @@
     <joint
       name="${end}_${side}_wheel_to_${end}_${side}_roller11"
-      type="continuous">
+      type="fixed">
       <origin
         xyz="0.015406 -0.01515 -0.066157"
@@ -744,7 +712,4 @@
       <child
         link="${end}_${side}_roller11" />
-      <axis
-        xyz="0 0 1" />
-      <dynamics friction="0.1"/>
     </joint>
     <link
@@ -790,5 +755,5 @@
     <joint
       name="${end}_${side}_wheel_to_${end}_${side}_roller12"
-      type="continuous">
+      type="fixed">
       <origin
         xyz="-0.012835 -0.01515 -0.066704"
@@ -798,7 +763,4 @@
       <child
         link="${end}_${side}_roller12" />
-      <axis
-        xyz="0 0 1" />
-      <dynamics friction="0.1"/>
     </joint>
     <link
@@ -844,5 +806,5 @@
     <joint
       name="${end}_${side}_wheel_to_${end}_${side}_roller13"
-      type="continuous">
+      type="fixed">
       <origin
         xyz="-0.038856 -0.01515 -0.055716"
@@ -852,7 +814,4 @@
       <child
         link="${end}_${side}_roller13" />
-      <axis
-        xyz="0 0 1" />
-      <dynamics friction="0.1"/>
     </joint>
     <link
@@ -898,5 +857,5 @@
     <joint
       name="${end}_${side}_wheel_to_${end}_${side}_roller14"
-      type="continuous">
+      type="fixed">
       <origin
         xyz="-0.058159 -0.01515 -0.035095"
@@ -906,7 +865,4 @@
       <child
         link="${end}_${side}_roller14" />
-      <axis
-        xyz="0 0 1" />
-      <dynamics friction="0.1"/>
     </joint>
     <link
@@ -952,5 +908,5 @@
     <joint
       name="${end}_${side}_wheel_to_${end}_${side}_roller15"
-      type="continuous">
+      type="fixed">
       <origin
         xyz="-0.0674050504299177 -0.0151497403158722 -0.00840608812639412"
@@ -960,7 +916,4 @@
       <child
         link="${end}_${side}_roller15" />
-      <axis
-        xyz="0 0 1" />
-      <dynamics friction="0.1"/>
     </joint>
   </xacro:macro>

File: linorobot2_description/urdf/mech/mecanum_wheel_right_fixed.urdf.xacro (robot description, xacro)
@@ -41,9 +41,8 @@
       </collision>
     </link>
-    <joint name="base_link_to_${end}_${side}_wheel" type="continuous">
+    <joint name="base_link_to_${end}_${side}_wheel" type="fixed">
       <origin xyz="${pos_x} ${pos_y} 0"  rpy="0 0 0" />
       <parent link="base_link" />
       <child link="${end}_${side}_wheel" />
-      <axis xyz="0 1 0" />
     </joint>
     <link
@@ -248,5 +247,5 @@
     <joint
       name="${end}_${side}_wheel_to_${end}_${side}_roller1"
-      type="continuous">
+      type="fixed">
       <origin
         xyz="0.0513105165568448 -0.0151129693198936 0.0444755356274741"
@@ -256,7 +255,4 @@
       <child
         link="${end}_${side}_roller1" />
-      <axis
-        xyz="0 0 1" />
-      <dynamics friction="0.1"/>
     </joint>
     <link
@@ -302,5 +298,5 @@
     <joint
       name="${end}_${side}_wheel_to_${end}_${side}_roller2"
-      type="continuous">
+      type="fixed">
       <origin
         xyz="0.0287846592696844 -0.0151129693198959 0.0615002908075162"
@@ -310,7 +306,4 @@
       <child
         link="${end}_${side}_roller2" />
-      <axis
-        xyz="0 0 1" />
-      <dynamics friction="0.1"/>
     </joint>
     <link
@@ -356,5 +349,5 @@
     <joint
       name="${end}_${side}_wheel_to_${end}_${side}_roller3"
-      type="continuous">
+      type="fixed">
       <origin
         xyz="0.00128167289437567 -0.0151129693198984 0.0678910869943366"
@@ -364,7 +357,4 @@
       <child
         link="${end}_${side}_roller3" />
-      <axis
-        xyz="0 0 1" />
-      <dynamics friction="0.1"/>
     </joint>
     <link
@@ -410,5 +400,5 @@
     <joint
       name="${end}_${side}_wheel_to_${end}_${side}_roller4"
-      type="continuous">
+      type="fixed">
       <origin
         xyz="-0.0264429263680024 -0.0151129693199014 0.062542897468674"
@@ -418,7 +408,4 @@
       <child
         link="${end}_${side}_roller4" />
-      <axis
-        xyz="0 0 1" />
-      <dynamics friction="0.1"/>
     </joint>
     <link
@@ -464,5 +451,5 @@
     <joint
       name="${end}_${side}_wheel_to_${end}_${side}_roller5"
-      type="continuous">
+      type="fixed">
       <origin
         xyz="-0.0495953034349089 -0.0151129693199047 0.0463804727862918"
@@ -472,7 +459,4 @@
       <child
         link="${end}_${side}_roller5" />
-      <axis
-        xyz="0 0 1" />
-      <dynamics friction="0.1"/>
     </joint>
     <link
@@ -518,5 +502,5 @@
     <joint
       name="${end}_${side}_wheel_to_${end}_${side}_roller6"
-      type="continuous">
+      type="fixed">
       <origin
         xyz="-0.0641722019787319 -0.0151129693199074 0.0221984430057918"
@@ -526,7 +510,4 @@
       <child
         link="${end}_${side}_roller6" />
-      <axis
-        xyz="0 0 1" />
-      <dynamics friction="0.1"/>
     </joint>
     <link
@@ -572,5 +553,5 @@
     <joint
       name="${end}_${side}_wheel_to_${end}_${side}_roller7"
-      type="continuous">
+      type="fixed">
       <origin
         xyz="-0.0676531438142786 -0.0151129693199092 -0.0058218992369328"
@@ -580,7 +561,4 @@
       <child
         link="${end}_${side}_roller7" />
-      <axis
-        xyz="0 0 1" />
-      <dynamics friction="0.1"/>
     </joint>
     <link
@@ -626,5 +604,5 @@
     <joint
       name="${end}_${side}_wheel_to_${end}_${side}_roller8"
-      type="continuous">
+      type="fixed">
       <origin
         xyz="-0.0594362424748194 -0.0151129693199101 -0.0328355822112983"
@@ -634,7 +612,4 @@
       <child
         link="${end}_${side}_roller8" />
-      <axis
-        xyz="0 0 1" />
-      <dynamics friction="0.1"/>
     </joint>
     <link
@@ -680,5 +655,5 @@
     <joint
       name="${end}_${side}_wheel_to_${end}_${side}_roller9"
-      type="continuous">
+      type="fixed">
       <origin
         xyz="-0.0409422748501527 -0.015112969319909 -0.0541716947194296"
@@ -688,7 +663,4 @@
       <child
         link="${end}_${side}_roller9" />
-      <axis
-        xyz="0 0 1" />
-      <dynamics friction="0.1"/>
     </joint>
     <link
@@ -734,5 +706,5 @@
     <joint
       name="${end}_${side}_wheel_to_${end}_${side}_roller10"
-      type="continuous">
+      type="fixed">
       <origin
         xyz="-0.0153690159550034 -0.0151129693199065 -0.0661410290761748"
@@ -742,7 +714,4 @@
       <child
         link="${end}_${side}_roller10" />
-      <axis
-        xyz="0 0 1" />
-      <dynamics friction="0.1"/>
     </joint>
     <link
@@ -788,5 +757,5 @@
     <joint
       name="${end}_${side}_wheel_to_${end}_${side}_roller11"
-      type="continuous">
+      type="fixed">
       <origin
         xyz="0.0128616854218928 -0.0151129693199038 -0.0666739786332639"
@@ -796,7 +765,4 @@
       <child
         link="${end}_${side}_roller11" />
-      <axis
-        xyz="0 0 1" />
-      <dynamics friction="0.1"/>
     </joint>
     <link
@@ -842,5 +808,5 @@
     <joint
       name="${end}_${side}_wheel_to_${end}_${side}_roller12"
-      type="continuous">
+      type="fixed">
       <origin
         xyz="0.0388684845445997 -0.0151129693199006 -0.0556783915705813"
@@ -850,7 +816,4 @@
       <child
         link="${end}_${side}_roller12" />
-      <axis
-        xyz="0 0 1" />
-      <dynamics friction="0.1"/>
     </joint>
     <link
@@ -896,5 +859,5 @@
     <joint
       name="${end}_${side}_wheel_to_${end}_${side}_roller13"
-      type="continuous">
+      type="fixed">
       <origin
         xyz="0.0581545695804492 -0.0151129693198971 -0.0350555047830372"
@@ -904,7 +867,4 @@
       <child
         link="${end}_${side}_roller13" />
-      <axis
-        xyz="0 0 1" />
-      <dynamics friction="0.1"/>
     </joint>
     <link
@@ -950,5 +910,5 @@
     <joint
       name="${end}_${side}_wheel_to_${end}_${side}_roller14"
-      type="continuous">
+      type="fixed">
       <origin
         xyz="0.0673852012181607 -0.0151129693198943 -0.00837120274924246"
@@ -958,7 +918,4 @@
       <child
         link="${end}_${side}_roller14" />
-      <axis
-        xyz="0 0 1" />
-      <dynamics friction="0.1"/>
     </joint>
     <link
@@ -1004,5 +961,5 @@
     <joint
       name="${end}_${side}_wheel_to_${end}_${side}_roller15"
-      type="continuous">
+      type="fixed">
       <origin
         xyz="0.0649643193899178 -0.0151129693198934 0.0197605562898849"
@@ -1012,7 +969,4 @@
       <child
         link="${end}_${side}_roller15" />
-      <axis
-        xyz="0 0 1" />
-      <dynamics friction="0.1"/>
     </joint>
   </xacro:macro>
