Commit message: Tried adding wheels as fixed single body entities, but FPS still dropped hard. Going without wheels for now

File: linorobot2_description/urdf/mech/mecanum_wheel_left_fixed.urdf.xacro (robot description, xacro)
@@ -1,5 +1,6 @@
 <?xml version="1.0"?>
 <robot xmlns:xacro="http://ros.org/wiki/xacro">
-  <xacro:macro name="mecanum_wheel_left" params="side end radius width pos_x pos_y pos_z mass">
+  <xacro:include filename="$(find linorobot2_description)/urdf/mech/roller_left.urdf.xacro" />
+  <xacro:macro name="mecanum_wheel_left" params="side end pos_x pos_y">
     <link name="${end}_${side}_wheel">
       <inertial>
@@ -23,5 +24,5 @@
         <geometry>
           <mesh
-            filename="package://linorobot2_description/mecanum_wheel_left/meshes/base_link.STL" />
+            filename="package://linorobot2_description/mecanum_wheel_left/meshes/fixed_wheel.STL" />
         </geometry>
         <material
@@ -37,5 +38,5 @@
         <geometry>
           <mesh
-            filename="package://linorobot2_description/mecanum_wheel_left/meshes/base_link.STL" />
+            filename="package://linorobot2_description/mecanum_wheel_left/meshes/fixed_wheel.STL" />
         </geometry>
       </collision>
@@ -46,875 +47,4 @@
       <child link="${end}_${side}_wheel" />
     </joint>
-    <link
-      name="${end}_${side}_plate1">
-      <inertial>
-        <origin
-          xyz="8.83119736279022E-16 3.33301269118141E-17 -0.000551568670724527"
-          rpy="0 0 0" />
-        <mass
-          value="0.0253986639693882" />
-        <inertia
-          ixx="4.21627753206923E-05"
-          ixy="1.3976043629696E-20"
-          ixz="-2.39458839321443E-21"
-          iyy="4.21627753206922E-05"
-          iyz="4.06169630282727E-21"
-          izz="8.39719993847474E-05" />
-      </inertial>
-      <visual>
-        <origin
-          xyz="0 0 0"
-          rpy="0 0 0" />
-        <geometry>
-          <mesh
-            filename="package://linorobot2_description/mecanum_wheel_left/meshes/plate1.STL" />
-        </geometry>
-        <material
-          name="">
-          <color
-            rgba="0.650980392156863 0.619607843137255 0.588235294117647 1" />
-        </material>
-      </visual>
-      <collision>
-        <origin
-          xyz="0 0 0"
-          rpy="0 0 0" />
-        <geometry>
-          <mesh
-            filename="package://linorobot2_description/mecanum_wheel_left/meshes/plate1.STL" />
-        </geometry>
-      </collision>
-    </link>
-    <joint
-      name="${end}_${side}_wheel_to_${end}_${side}_plate1"
-      type="fixed">
-      <origin
-        xyz="0 0.023114 0"
-        rpy="-1.5708 0.03287 0" />
-      <parent
-        link="${end}_${side}_wheel" />
-      <child
-        link="${end}_${side}_plate1" />
-      <axis
-        xyz="0 0 0" />
-    </joint>
-    <link
-      name="${end}_${side}_plate2">
-      <inertial>
-        <origin
-          xyz="-1.10651810076925E-15 8.09386876632109E-17 -0.000551568670724527"
-          rpy="0 0 0" />
-        <mass
-          value="0.0253986639693882" />
-        <inertia
-          ixx="4.21627753206924E-05"
-          ixy="1.65171424714589E-20"
-          ixz="4.28643950323039E-22"
-          iyy="4.21627753206923E-05"
-          iyz="2.75305456980319E-21"
-          izz="8.39719993847476E-05" />
-      </inertial>
-      <visual>
-        <origin
-          xyz="0 0 0"
-          rpy="0 0 0" />
-        <geometry>
-          <mesh
-            filename="package://linorobot2_description/mecanum_wheel_left/meshes/plate2.STL" />
-        </geometry>
-        <material
-          name="">
-          <color
-            rgba="0.650980392156863 0.619607843137255 0.588235294117647 1" />
-        </material>
-      </visual>
-      <collision>
-        <origin
-          xyz="0 0 0"
-          rpy="0 0 0" />
-        <geometry>
-          <mesh
-            filename="package://linorobot2_description/mecanum_wheel_left/meshes/plate2.STL" />
-        </geometry>
-      </collision>
-    </link>
-    <joint
-      name="${end}_${side}_wheel_to_${end}_${side}_plate2"
-      type="fixed">
-      <origin
-        xyz="0 -0.023114 0"
-        rpy="-1.5707963267949 0.0335546833724646 -3.14159265358979" />
-      <parent
-        link="${end}_${side}_wheel" />
-      <child
-        link="${end}_${side}_plate2" />
-      <axis
-        xyz="0 0 0" />
-    </joint>
-    <link
-      name="${end}_${side}_roller1">
-      <inertial>
-        <origin
-          xyz="5.96744875736022E-16 -1.24475083018716E-14 -0.0215899999999933"
-          rpy="0 0 0" />
-        <mass
-          value="0.00499543658848208" />
-        <inertia
-          ixx="8.99919949242919E-07"
-          ixy="3.97046694025453E-23"
-          ixz="9.81863387100444E-22"
-          iyy="8.9991994924288E-07"
-          iyz="-8.0163727523739E-19"
-          izz="3.31951561004127E-07" />
-      </inertial>
-      <visual>
-        <origin
-          xyz="0 0 0"
-          rpy="0 0 0" />
-        <geometry>
-          <mesh
-            filename="package://linorobot2_description/mecanum_wheel_left/meshes/roller1.STL" />
-        </geometry>
-        <material
-          name="">
-          <color
-            rgba="0.752941176470588 0.752941176470588 0.752941176470588 1" />
-        </material>
-      </visual>
-      <collision>
-        <origin
-          xyz="0 0 0"
-          rpy="0 0 0" />
-        <geometry>
-          <mesh
-            filename="package://linorobot2_description/mecanum_wheel_left/meshes/roller1.STL" />
-        </geometry>
-      </collision>
-    </link>
-    <joint
-      name="${end}_${side}_wheel_to_${end}_${side}_roller1"
-      type="fixed">
-      <origin
-        xyz="-0.064997 -0.01515 0.019737"
-        rpy="2.3375 0.48899 -0.038445" />
-      <parent
-        link="${end}_${side}_wheel" />
-      <child
-        link="${end}_${side}_roller1" />
-    </joint>
-    <link
-      name="${end}_${side}_roller2">
-      <inertial>
-        <origin
-          xyz="5.96744875736022E-16 -1.24475083018716E-14 -0.0215899999999933"
-          rpy="0 0 0" />
-        <mass
-          value="0.00499543658848208" />
-        <inertia
-          ixx="8.99919949242919E-07"
-          ixy="3.97046694025453E-23"
-          ixz="9.81863387100444E-22"
-          iyy="8.9991994924288E-07"
-          iyz="-8.0163727523739E-19"
-          izz="3.31951561004127E-07" />
-      </inertial>
-      <visual>
-        <origin
-          xyz="0 0 0"
-          rpy="0 0 0" />
-        <geometry>
-          <mesh
-            filename="package://linorobot2_description/mecanum_wheel_left/meshes/roller2.STL" />
-        </geometry>
-        <material
-          name="">
-          <color
-            rgba="0.752941176470588 0.752941176470588 0.752941176470588 1" />
-        </material>
-      </visual>
-      <collision>
-        <origin
-          xyz="0 0 0"
-          rpy="0 0 0" />
-        <geometry>
-          <mesh
-            filename="package://linorobot2_description/mecanum_wheel_left/meshes/roller2.STL" />
-        </geometry>
-      </collision>
-    </link>
-    <joint
-      name="${end}_${side}_wheel_to_${end}_${side}_roller2"
-      type="fixed">
-      <origin
-        xyz="-0.05135 -0.01515 0.044467"
-        rpy="2.3122 0.90744 -0.055132" />
-      <parent
-        link="${end}_${side}_wheel" />
-      <child
-        link="${end}_${side}_roller2" />
-    </joint>
-    <link
-      name="${end}_${side}_roller3">
-      <inertial>
-        <origin
-          xyz="5.96744875736022E-16 -1.24475083018716E-14 -0.0215899999999933"
-          rpy="0 0 0" />
-        <mass
-          value="0.00499543658848208" />
-        <inertia
-          ixx="8.99919949242919E-07"
-          ixy="3.97046694025453E-23"
-          ixz="9.81863387100444E-22"
-          iyy="8.9991994924288E-07"
-          iyz="-8.0163727523739E-19"
-          izz="3.31951561004127E-07" />
-      </inertial>
-      <visual>
-        <origin
-          xyz="0 0 0"
-          rpy="0 0 0" />
-        <geometry>
-          <mesh
-            filename="package://linorobot2_description/mecanum_wheel_left/meshes/roller3.STL" />
-        </geometry>
-        <material
-          name="">
-          <color
-            rgba="0.752941176470588 0.752941176470588 0.752941176470588 1" />
-        </material>
-      </visual>
-      <collision>
-        <origin
-          xyz="0 0 0"
-          rpy="0 0 0" />
-        <geometry>
-          <mesh
-            filename="package://linorobot2_description/mecanum_wheel_left/meshes/roller3.STL" />
-        </geometry>
-      </collision>
-    </link>
-    <joint
-      name="${end}_${side}_wheel_to_${end}_${side}_roller3"
-      type="fixed">
-      <origin
-        xyz="-0.028824 -0.01515 0.061508"
-        rpy="2.22 1.3248 -0.13976" />
-      <parent
-        link="${end}_${side}_wheel" />
-      <child
-        link="${end}_${side}_roller3" />
-    </joint>
-    <link
-      name="${end}_${side}_roller4">
-      <inertial>
-        <origin
-          xyz="5.96744875736022E-16 -1.24475083018716E-14 -0.0215899999999933"
-          rpy="0 0 0" />
-        <mass
-          value="0.00499543658848208" />
-        <inertia
-          ixx="8.99919949242919E-07"
-          ixy="3.97046694025453E-23"
-          ixz="9.81863387100444E-22"
-          iyy="8.9991994924288E-07"
-          iyz="-8.0163727523739E-19"
-          izz="3.31951561004127E-07" />
-      </inertial>
-      <visual>
-        <origin
-          xyz="0 0 0"
-          rpy="0 0 0" />
-        <geometry>
-          <mesh
-            filename="package://linorobot2_description/mecanum_wheel_left/meshes/roller4.STL" />
-        </geometry>
-        <material
-          name="">
-          <color
-            rgba="0.752941176470588 0.752941176470588 0.752941176470588 1" />
-        </material>
-      </visual>
-      <collision>
-        <origin
-          xyz="0 0 0"
-          rpy="0 0 0" />
-        <geometry>
-          <mesh
-            filename="package://linorobot2_description/mecanum_wheel_left/meshes/roller4.STL" />
-        </geometry>
-      </collision>
-    </link>
-    <joint
-      name="${end}_${side}_wheel_to_${end}_${side}_roller4"
-      type="fixed">
-      <origin
-        xyz="-0.0013143 -0.01515 0.067914"
-        rpy="-0.59653 1.3924 -2.9492" />
-      <parent
-        link="${end}_${side}_wheel" />
-      <child
-        link="${end}_${side}_roller4" />
-    </joint>
-    <link
-      name="${end}_${side}_roller5">
-      <inertial>
-        <origin
-          xyz="5.96744875736022E-16 -1.24475083018716E-14 -0.0215899999999933"
-          rpy="0 0 0" />
-        <mass
-          value="0.00499543658848208" />
-        <inertia
-          ixx="8.99919949242919E-07"
-          ixy="3.97046694025453E-23"
-          ixz="9.81863387100444E-22"
-          iyy="8.9991994924288E-07"
-          iyz="-8.0163727523739E-19"
-          izz="3.31951561004127E-07" />
-      </inertial>
-      <visual>
-        <origin
-          xyz="0 0 0"
-          rpy="0 0 0" />
-        <geometry>
-          <mesh
-            filename="package://linorobot2_description/mecanum_wheel_left/meshes/roller5.STL" />
-        </geometry>
-        <material
-          name="">
-          <color
-            rgba="0.752941176470588 0.752941176470588 0.752941176470588 1" />
-        </material>
-      </visual>
-      <collision>
-        <origin
-          xyz="0 0 0"
-          rpy="0 0 0" />
-        <geometry>
-          <mesh
-            filename="package://linorobot2_description/mecanum_wheel_left/meshes/roller5.STL" />
-        </geometry>
-      </collision>
-    </link>
-    <joint
-      name="${end}_${side}_wheel_to_${end}_${side}_roller5"
-      type="fixed">
-      <origin
-        xyz="0.026423 -0.01515 0.062578"
-        rpy="-0.73578 0.97593 -3.081" />
-      <parent
-        link="${end}_${side}_wheel" />
-      <child
-        link="${end}_${side}_roller5" />
-    </joint>
-    <link
-      name="${end}_${side}_roller6">
-      <inertial>
-        <origin
-          xyz="5.96744875736022E-16 -1.24475083018716E-14 -0.0215899999999933"
-          rpy="0 0 0" />
-        <mass
-          value="0.00499543658848208" />
-        <inertia
-          ixx="8.99919949242919E-07"
-          ixy="3.97046694025453E-23"
-          ixz="9.81863387100444E-22"
-          iyy="8.9991994924288E-07"
-          iyz="-8.0163727523739E-19"
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