Commit message: Tried adding wheels as fixed single body entities, but FPS still dropped hard. Going without wheels for now

File: linorobot2_description/urdf/mech/mecanum_wheel_right_fixed.urdf.xacro (robot description, xacro)
@@ -1,5 +1,5 @@
 <?xml version="1.0"?>
 <robot xmlns:xacro="http://ros.org/wiki/xacro">
-  <xacro:macro name="mecanum_wheel_right" params="side end radius width pos_x pos_y pos_z mass">
+  <xacro:macro name="mecanum_wheel_right" params="side end pos_x pos_y">
     <link name="${end}_${side}_wheel">
       <inertial>
@@ -23,5 +23,5 @@
         <geometry>
           <mesh
-            filename="package://linorobot2_description/mecanum_wheel_right/meshes/base_link.STL" />
+            filename="package://linorobot2_description/mecanum_wheel_right/meshes/fixed_wheel.STL" />
         </geometry>
         <material
@@ -37,5 +37,5 @@
         <geometry>
           <mesh
-            filename="package://linorobot2_description/mecanum_wheel_right/meshes/base_link.STL" />
+            filename="package://linorobot2_description/mecanum_wheel_right/meshes/fixed_wheel.STL" />
         </geometry>
       </collision>
@@ -46,928 +46,4 @@
       <child link="${end}_${side}_wheel" />
     </joint>
-    <link
-      name="${end}_${side}_drum">
-      <inertial>
-      <origin
-        xyz="0.0136209233699844 6.56957443528167E-16 -1.48512976903392E-15"
-        rpy="0 0 0" />
-      <mass
-        value="0.0396439871820506" />
-      <inertia
-        ixx="7.1054120055567E-05"
-        ixy="1.62690471844664E-18"
-        ixz="-3.70636817664487E-18"
-        iyy="3.76805204137311E-05"
-        iyz="1.0973915143622E-20"
-        izz="3.76805204137311E-05" />
-    </inertial>
-      <visual>
-        <origin
-          xyz="0 0 0"
-          rpy="0 0 0" />
-        <geometry>
-          <mesh
-            filename="package://linorobot2_description/mecanum_wheel_right/meshes/drum.STL" />
-        </geometry>
-        <material
-          name="">
-          <color
-            rgba="0.898039215686275 0.917647058823529 0.929411764705882 1" />
-        </material>
-      </visual>
-      <collision>
-        <origin
-          xyz="0 0 0"
-          rpy="0 0 0" />
-        <geometry>
-          <mesh
-            filename="package://linorobot2_description/mecanum_wheel_right/meshes/drum.STL" />
-        </geometry>
-      </collision>
-    </link>
-    <joint
-      name="${end}_${side}_wheel_to_drum"
-      type="fixed">
-      <origin
-        xyz="0 0 0"
-        rpy="1.5707963267949 0 -1.5707963267949" />
-      <parent
-        link="${end}_${side}_wheel" />
-      <child
-        link="${end}_${side}_drum" />
-      <axis
-        xyz="0 0 0" />
-    </joint>
-    <link
-      name="${end}_${side}_plate1">
-      <inertial>
-      <origin
-        xyz="-0.00283756867072453 8.89413056967719E-16 2.68096171575045E-15"
-        rpy="0 0 0" />
-      <mass
-        value="0.0253986639693881" />
-      <inertia
-        ixx="8.39719993847471E-05"
-        ixy="1.90079838330856E-18"
-        ixz="4.7133202434868E-18"
-        iyy="4.21627753206921E-05"
-        iyz="-1.48230765769502E-20"
-        izz="4.21627753206921E-05" />
-    </inertial>
-      <visual>
-        <origin
-          xyz="0 0 0"
-          rpy="0 0 0" />
-        <geometry>
-          <mesh
-            filename="package://linorobot2_description/mecanum_wheel_right/meshes/plate1.STL" />
-        </geometry>
-        <material
-          name="">
-          <color
-            rgba="0.752941176470588 0.752941176470588 0.752941176470588 1" />
-        </material>
-      </visual>
-      <collision>
-        <origin
-          xyz="0 0 0"
-          rpy="0 0 0" />
-        <geometry>
-          <mesh
-            filename="package://linorobot2_description/mecanum_wheel_right/meshes/plate1.STL" />
-        </geometry>
-      </collision>
-    </link>
-    <joint
-      name="${end}_${side}_wheel_to_${end}_${side}_plate1"
-      type="fixed">
-      <origin
-        xyz="0 0.0254 0"
-        rpy="-1.60435101016735 0 1.5707963267949" />
-      <parent
-        link="${end}_${side}_wheel" />
-      <child
-        link="${end}_${side}_plate1" />
-      <axis
-        xyz="0 0 0" />
-    </joint>
-    <link
-      name="${end}_${side}_plate2">
-      <inertial>
-      <origin
-        xyz="-0.00283756867072453 -9.8249688244021E-17 5.89771118826868E-17"
-        rpy="0 0 0" />
-      <mass
-        value="0.0253986639693881" />
-      <inertia
-        ixx="8.39719993847471E-05"
-        ixy="-9.13983660820293E-21"
-        ixz="5.31128745957199E-22"
-        iyy="4.2162775320692E-05"
-        iyz="1.59877468794249E-20"
-        izz="4.21627753206921E-05" />
-    </inertial>
-      <visual>
-        <origin
-          xyz="0 0 0"
-          rpy="0 0 0" />
-        <geometry>
-          <mesh
-            filename="package://linorobot2_description/mecanum_wheel_right/meshes/plate2.STL" />
-        </geometry>
-        <material
-          name="">
-          <color
-            rgba="0.752941176470588 0.752941176470588 0.752941176470588 1" />
-        </material>
-      </visual>
-      <collision>
-        <origin
-          xyz="0 0 0"
-          rpy="0 0 0" />
-        <geometry>
-          <mesh
-            filename="package://linorobot2_description/mecanum_wheel_right/meshes/plate2.STL" />
-        </geometry>
-      </collision>
-    </link>
-    <joint
-      name="${end}_${side}_wheel_to_${end}_${side}_plate2"
-      type="fixed">
-      <origin
-        xyz="0 -0.0254 0"
-        rpy="1.60435101016734 0 -1.5707963267949" />
-      <parent
-        link="${end}_${side}_wheel" />
-      <child
-        link="${end}_${side}_plate2" />
-      <axis
-        xyz="0 0 0" />
-    </joint>
-    <link
-      name="${end}_${side}_roller1">
-      <inertial>
-      <origin
-        xyz="5.82867087928207E-16 3.51108031537706E-15 -0.0215899999999933"
-        rpy="0 0 0" />
-      <mass
-        value="0.00499543658848254" />
-      <inertia
-        ixx="8.99919949255961E-07"
-        ixy="0"
-        ixz="7.14684049245816E-22"
-        iyy="8.999199492559E-07"
-        iyz="-8.01670362461892E-19"
-        izz="3.31951561028667E-07" />
-    </inertial>
-      <visual>
-        <origin
-          xyz="0 0 0"
-          rpy="0 0 0" />
-        <geometry>
-          <mesh
-            filename="package://linorobot2_description/mecanum_wheel_right/meshes/roller1.STL" />
-        </geometry>
-        <material
-          name="">
-          <color
-            rgba="0.752941176470588 0.752941176470588 0.752941176470588 1" />
-        </material>
-      </visual>
-      <collision>
-        <origin
-          xyz="0 0 0"
-          rpy="0 0 0" />
-        <geometry>
-          <mesh
-            filename="package://linorobot2_description/mecanum_wheel_right/meshes/roller1.STL" />
-        </geometry>
-      </collision>
-    </link>
-    <joint
-      name="${end}_${side}_wheel_to_${end}_${side}_roller1"
-      type="fixed">
-      <origin
-        xyz="0.0513105165568448 -0.0151129693198936 0.0444755356274741"
-        rpy="-2.36778917303694 -0.95454994461673 -1.76416393166909" />
-      <parent
-        link="${end}_${side}_wheel" />
-      <child
-        link="${end}_${side}_roller1" />
-    </joint>
-    <link
-      name="${end}_${side}_roller2">
-      <inertial>
-      <origin
-        xyz="5.82867087928207E-16 3.51108031537706E-15 -0.0215899999999933"
-        rpy="0 0 0" />
-      <mass
-        value="0.00499543658848254" />
-      <inertia
-        ixx="8.99919949255961E-07"
-        ixy="0"
-        ixz="7.14684049245816E-22"
-        iyy="8.999199492559E-07"
-        iyz="-8.01670362461892E-19"
-        izz="3.31951561028667E-07" />
-    </inertial>
-      <visual>
-        <origin
-          xyz="0 0 0"
-          rpy="0 0 0" />
-        <geometry>
-          <mesh
-            filename="package://linorobot2_description/mecanum_wheel_right/meshes/roller2.STL" />
-        </geometry>
-        <material
-          name="">
-          <color
-            rgba="0.752941176470588 0.752941176470588 0.752941176470588 1" />
-        </material>
-      </visual>
-      <collision>
-        <origin
-          xyz="0 0 0"
-          rpy="0 0 0" />
-        <geometry>
-          <mesh
-            filename="package://linorobot2_description/mecanum_wheel_right/meshes/roller2.STL" />
-        </geometry>
-      </collision>
-    </link>
-    <joint
-      name="${end}_${side}_wheel_to_${end}_${side}_roller2"
-      type="fixed">
-      <origin
-        xyz="0.0287846592696844 -0.0151129693198959 0.0615002908075162"
-        rpy="-1.77439072812908 -0.775855866169197 -2.22324127737972" />
-      <parent
-        link="${end}_${side}_wheel" />
-      <child
-        link="${end}_${side}_roller2" />
-    </joint>
-    <link
-      name="${end}_${side}_roller3">
-      <inertial>
-      <origin
-        xyz="5.82867087928207E-16 3.51108031537706E-15 -0.0215899999999933"
-        rpy="0 0 0" />
-      <mass
-        value="0.00499543658848254" />
-      <inertia
-        ixx="8.99919949255961E-07"
-        ixy="0"
-        ixz="7.14684049245816E-22"
-        iyy="8.999199492559E-07"
-        iyz="-8.01670362461892E-19"
-        izz="3.31951561028667E-07" />
-    </inertial>
-      <visual>
-        <origin
-          xyz="0 0 0"
-          rpy="0 0 0" />
-        <geometry>
-          <mesh
-            filename="package://linorobot2_description/mecanum_wheel_right/meshes/roller3.STL" />
-        </geometry>
-        <material
-          name="">
-          <color
-            rgba="0.752941176470588 0.752941176470588 0.752941176470588 1" />
-        </material>
-      </visual>
-      <collision>
-        <origin
-          xyz="0 0 0"
-          rpy="0 0 0" />
-        <geometry>
-          <mesh
-            filename="package://linorobot2_description/mecanum_wheel_right/meshes/roller3.STL" />
-        </geometry>
-      </collision>
-    </link>
-    <joint
-      name="${end}_${side}_wheel_to_${end}_${side}_roller3"
-      type="fixed">
-      <origin
-        xyz="0.00128167289437567 -0.0151129693198984 0.0678910869943366"
-        rpy="-1.40103696999546 -0.48194994387805 -2.44694050545059" />
-      <parent
-        link="${end}_${side}_wheel" />
-      <child
-        link="${end}_${side}_roller3" />
-    </joint>
-    <link
-      name="${end}_${side}_roller4">
-      <inertial>
-      <origin
-        xyz="5.82867087928207E-16 3.51108031537706E-15 -0.0215899999999933"
-        rpy="0 0 0" />
-      <mass
-        value="0.00499543658848254" />
-      <inertia
-        ixx="8.99919949255961E-07"
-        ixy="0"
-        ixz="7.14684049245816E-22"
-        iyy="8.999199492559E-07"
-        iyz="-8.01670362461892E-19"
-        izz="3.31951561028667E-07" />
-    </inertial>
-      <visual>
-        <origin
-          xyz="0 0 0"
-          rpy="0 0 0" />
-        <geometry>
-          <mesh
-            filename="package://linorobot2_description/mecanum_wheel_right/meshes/roller4.STL" />
-        </geometry>
-        <material
-          name="">
-          <color
-            rgba="0.752941176470588 0.752941176470588 0.752941176470588 1" />
-        </material>
-      </visual>
-      <collision>
-        <origin
-          xyz="0 0 0"
-          rpy="0 0 0" />
-        <geometry>
-          <mesh
-            filename="package://linorobot2_description/mecanum_wheel_right/meshes/roller4.STL" />
-        </geometry>
-      </collision>
-    </link>
-    <joint
-      name="${end}_${side}_wheel_to_${end}_${side}_roller4"
-      type="fixed">
-      <origin
-        xyz="-0.0264429263680024 -0.0151129693199014 0.062542897468674"
-        rpy="-1.13469826196558 -0.147073422491862 -2.53094960861872" />
-      <parent
-        link="${end}_${side}_wheel" />
-      <child
-        link="${end}_${side}_roller4" />
-    </joint>
-    <link
-      name="${end}_${side}_roller5">
-      <inertial>
-      <origin
-        xyz="5.82867087928207E-16 3.51108031537706E-15 -0.0215899999999933"
-        rpy="0 0 0" />
-      <mass
-        value="0.00499543658848254" />
-      <inertia
-        ixx="8.99919949255961E-07"
-        ixy="0"
-        ixz="7.14684049245816E-22"
-        iyy="8.999199492559E-07"
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
File: linorobot2_description/urdf/robots/mecanum_libplanar.urdf.xacro (robot description, xacro)
@@ -8,5 +8,5 @@
   <xacro:include filename="$(find linorobot2_description)/urdf/mech/side_channel.urdf.xacro" />
   <xacro:include filename="$(find linorobot2_description)/urdf/robots/camera.urdf.xacro" />
-  <xacro:camera camera_pos="front" x="0.410335" y="0" z="0.0892"
+  <!-- <xacro:camera camera_pos="front" x="0.410335" y="0" z="0.0892"
                                    r_rs="-1.57" p_rs="0" yaw_rs="-1.57" />
   <xacro:camera camera_pos="left" x="0.0" y="0.247" z="0.089"
@@ -15,5 +15,5 @@
                                   r_rs="-1.57" p_rs="0" yaw_rs="1.57" />
   <xacro:camera camera_pos="right" x="0" y="-0.247" z="0.089"
-                                  r_rs="-1.57" p_rs="0" yaw_rs="3.14"/>
+                                  r_rs="-1.57" p_rs="0" yaw_rs="3.14"/> -->
   <gazebo>
     <plugin name="mecanum_wheel_mimic" filename="libgazebo_ros_planar_move.so">
@@ -54,44 +54,27 @@
     pos_y="-0.23653"
   />
-  <xacro:mecanum_wheel_left
+  <!-- <xacro:mecanum_wheel_left
     side="left"
     end="front"
-    radius="${wheel_radius}"
-    width="${wheel_width}"
     pos_x="${wheel_pos_x}"
     pos_y="${wheel_pos_y}"
-    pos_z="${wheel_pos_z}"
-    mass="${wheel_mass}"
   />
   <xacro:mecanum_wheel_right
     side="right"
     end="front"
-    radius="${wheel_radius}"
-    width="${wheel_width}"
     pos_x="${wheel_pos_x}"
     pos_y="${-wheel_pos_y}"
-    pos_z="${wheel_pos_z}"
-    mass="${wheel_mass}"
   />
-  <!-- Back wheels mechanum style swapped (left mecanum wheel goes on right side of robot, and vice versa) -->
   <xacro:mecanum_wheel_right
     side="left"
     end="rear"
-    radius="${wheel_radius}"
-    width="${wheel_width}"
     pos_x="${-wheel_pos_x}"
     pos_y="${wheel_pos_y}"
-    pos_z="${wheel_pos_z}"
-    mass="${wheel_mass}"
   />
   <xacro:mecanum_wheel_left
     side="right"
     end="rear"
-    radius="${wheel_radius}"
-    width="${wheel_width}"
     pos_x="${-wheel_pos_x}"
     pos_y="${-wheel_pos_y}"
-    pos_z="${wheel_pos_z}"
-    mass="${wheel_mass}"
-  />
+  /> -->
 </robot>
