Commit message: Added inertia tags back to robot links so that robot can be used in gazebo

File: linorobot2_description/urdf/mech/base.urdf.xacro (robot description, xacro)
@@ -8,5 +8,4 @@
         <geometry>
           <box size="${length} ${width} ${height}"/>
-          <!-- <mesh filename="" scale="0.001 0.001 0.001"/> -->
         </geometry>
         <material name="gray_base">
@@ -22,5 +21,6 @@
       <inertial>
         <origin xyz="0 0 0" rpy="0 0 0"/>
-        <mass value="${mass}"/>
+        <mass value="0"/>
+        <inertia ixx="0"  ixy="0"  ixz="0" iyy="0" iyz="0" izz="0" />
       </inertial>
     </link>

File: linorobot2_description/urdf/mech/end_channel.urdf.xacro (robot description, xacro)
@@ -17,5 +17,13 @@
       </collision>
       <inertial>
+        <origin xyz="0 0 0" rpy="0 0 0" />
         <mass value="5"/>
+        <inertia
+          ixx="0.1052"
+          ixy="0"
+          ixz="0"
+          iyy="0.0042"
+          iyz="0"
+          izz="0.1034" />
       </inertial>
     </link>

File: linorobot2_description/urdf/mech/mecanum_wheel_left.urdf.xacro (robot description, xacro)
@@ -8,6 +8,13 @@
           rpy="0 0 0" />
         <mass
-          value="0.25" />
-      </inertial>
+          value="0.039620820516108" />
+        <inertia
+          ixx="3.76577202480009E-05"
+          ixy="-1.07908308681007E-19"
+          ixz="3.89356499633093E-22"
+          iyy="7.10123305553507E-05"
+          iyz="-1.66085499471637E-18"
+          izz="3.76577202480009E-05" />
+    </inertial>
       <visual>
         <origin
@@ -44,7 +51,17 @@
       name="${end}_${side}_plate1">
       <inertial>
-        <mass
-          value="0.5" />
-      </inertial>
+        <origin
+          xyz="8.83119736279022E-16 3.33301269118141E-17 -0.000551568670724527"
+          rpy="0 0 0" />
+        <mass
+          value="0.0253986639693882" />
+        <inertia
+          ixx="4.21627753206923E-05"
+          ixy="1.3976043629696E-20"
+          ixz="-2.39458839321443E-21"
+          iyy="4.21627753206922E-05"
+          iyz="4.06169630282727E-21"
+          izz="8.39719993847474E-05" />
+    </inertial>
       <visual>
         <origin
@@ -87,6 +104,17 @@
       name="${end}_${side}_plate2">
       <inertial>
-        <mass value="0.5" />
-      </inertial>
+        <origin
+          xyz="-1.10651810076925E-15 8.09386876632109E-17 -0.000551568670724527"
+          rpy="0 0 0" />
+        <mass
+          value="0.0253986639693882" />
+        <inertia
+          ixx="4.21627753206924E-05"
+          ixy="1.65171424714589E-20"
+          ixz="4.28643950323039E-22"
+          iyy="4.21627753206923E-05"
+          iyz="2.75305456980319E-21"
+          izz="8.39719993847476E-05" />
+    </inertial>
       <visual>
         <origin
@@ -133,6 +161,13 @@
           rpy="0 0 0" />
         <mass
-          value="0.025" />
-      </inertial>
+          value="0.00499543658848208" />
+        <inertia
+          ixx="8.99919949242919E-07"
+          ixy="3.97046694025453E-23"
+          ixz="9.81863387100444E-22"
+          iyy="8.9991994924288E-07"
+          iyz="-8.0163727523739E-19"
+          izz="3.31951561004127E-07" />
+    </inertial>
       <visual>
         <origin
@@ -177,9 +212,16 @@
       <inertial>
         <origin
-          xyz="5.82867087928207E-16 -9.95687907123788E-15 -0.0215899999999933"
-          rpy="0 0 0" />
-        <mass
-          value="0.025" />
-      </inertial>
+          xyz="5.96744875736022E-16 -1.24475083018716E-14 -0.0215899999999933"
+          rpy="0 0 0" />
+        <mass
+          value="0.00499543658848208" />
+        <inertia
+          ixx="8.99919949242919E-07"
+          ixy="3.97046694025453E-23"
+          ixz="9.81863387100444E-22"
+          iyy="8.9991994924288E-07"
+          iyz="-8.0163727523739E-19"
+          izz="3.31951561004127E-07" />
+    </inertial>
       <visual>
         <origin
@@ -224,9 +266,16 @@
       <inertial>
         <origin
-          xyz="5.82867087928207E-16 -3.41003267290141E-15 -0.0215899999999933"
-          rpy="0 0 0" />
-        <mass
-          value="0.025" />
-      </inertial>
+          xyz="5.96744875736022E-16 -1.24475083018716E-14 -0.0215899999999933"
+          rpy="0 0 0" />
+        <mass
+          value="0.00499543658848208" />
+        <inertia
+          ixx="8.99919949242919E-07"
+          ixy="3.97046694025453E-23"
+          ixz="9.81863387100444E-22"
+          iyy="8.9991994924288E-07"
+          iyz="-8.0163727523739E-19"
+          izz="3.31951561004127E-07" />
+    </inertial>
       <visual>
         <origin
@@ -271,9 +320,16 @@
       <inertial>
         <origin
-          xyz="5.68989300120393E-16 -3.35365415993216E-15 -0.0215899999999933"
-          rpy="0 0 0" />
-        <mass
-          value="0.025" />
-      </inertial>
+          xyz="5.96744875736022E-16 -1.24475083018716E-14 -0.0215899999999933"
+          rpy="0 0 0" />
+        <mass
+          value="0.00499543658848208" />
+        <inertia
+          ixx="8.99919949242919E-07"
+          ixy="3.97046694025453E-23"
+          ixz="9.81863387100444E-22"
+          iyy="8.9991994924288E-07"
+          iyz="-8.0163727523739E-19"
+          izz="3.31951561004127E-07" />
+    </inertial>
       <visual>
         <origin
@@ -318,9 +374,16 @@
       <inertial>
         <origin
-          xyz="5.96744875736022E-16 2.4459601011273E-15 -0.0215899999999933"
-          rpy="0 0 0" />
-        <mass
-          value="0.025" />
-      </inertial>
+          xyz="5.96744875736022E-16 -1.24475083018716E-14 -0.0215899999999933"
+          rpy="0 0 0" />
+        <mass
+          value="0.00499543658848208" />
+        <inertia
+          ixx="8.99919949242919E-07"
+          ixy="3.97046694025453E-23"
+          ixz="9.81863387100444E-22"
+          iyy="8.9991994924288E-07"
+          iyz="-8.0163727523739E-19"
+          izz="3.31951561004127E-07" />
+    </inertial>
       <visual>
         <origin
@@ -365,9 +428,16 @@
       <inertial>
         <origin
-          xyz="5.82867087928207E-16 -7.52392939618041E-15 -0.0215899999999933"
-          rpy="0 0 0" />
-        <mass
-          value="0.025" />
-      </inertial>
+          xyz="5.96744875736022E-16 -1.24475083018716E-14 -0.0215899999999933"
+          rpy="0 0 0" />
+        <mass
+          value="0.00499543658848208" />
+        <inertia
+          ixx="8.99919949242919E-07"
+          ixy="3.97046694025453E-23"
+          ixz="9.81863387100444E-22"
+          iyy="8.9991994924288E-07"
+          iyz="-8.0163727523739E-19"
+          izz="3.31951561004127E-07" />
+    </inertial>
       <visual>
         <origin
@@ -412,9 +482,16 @@
       <inertial>
         <origin
-          xyz="5.82867087928207E-16 -3.4109000346394E-15 -0.0215899999999933"
-          rpy="0 0 0" />
-        <mass
-          value="0.025" />
-      </inertial>
+          xyz="5.96744875736022E-16 -1.24475083018716E-14 -0.0215899999999933"
+          rpy="0 0 0" />
+        <mass
+          value="0.00499543658848208" />
+        <inertia
+          ixx="8.99919949242919E-07"
+          ixy="3.97046694025453E-23"
+          ixz="9.81863387100444E-22"
+          iyy="8.9991994924288E-07"
+          iyz="-8.0163727523739E-19"
+          izz="3.31951561004127E-07" />
+    </inertial>
       <visual>
         <origin
@@ -459,9 +536,16 @@
       <inertial>
         <origin
-          xyz="5.82867087928207E-16 -1.76421377506841E-15 -0.0215899999999933"
-          rpy="0 0 0" />
-        <mass
-          value="0.025" />
-      </inertial>
+          xyz="5.96744875736022E-16 -1.24475083018716E-14 -0.0215899999999933"
+          rpy="0 0 0" />
+        <mass
+          value="0.00499543658848208" />
+        <inertia
+          ixx="8.99919949242919E-07"
+          ixy="3.97046694025453E-23"
+          ixz="9.81863387100444E-22"
+          iyy="8.9991994924288E-07"
+          iyz="-8.0163727523739E-19"
+          izz="3.31951561004127E-07" />
+    </inertial>
       <visual>
         <origin
@@ -506,9 +590,16 @@
       <inertial>
         <origin
-          xyz="5.82867087928207E-16 -5.1013880619788E-15 -0.0215899999999933"
-          rpy="0 0 0" />
-        <mass
-          value="0.025" />
-      </inertial>
+          xyz="5.96744875736022E-16 -1.24475083018716E-14 -0.0215899999999933"
+          rpy="0 0 0" />
+        <mass
+          value="0.00499543658848208" />
+        <inertia
+          ixx="8.99919949242919E-07"
+          ixy="3.97046694025453E-23"
+          ixz="9.81863387100444E-22"
+          iyy="8.9991994924288E-07"
+          iyz="-8.0163727523739E-19"
+          izz="3.31951561004127E-07" />
+    </inertial>
       <visual>
         <origin
@@ -553,9 +644,16 @@
       <inertial>
         <origin
-          xyz="5.96744875736022E-16 -6.51952450358984E-15 -0.0215899999999933"
-          rpy="0 0 0" />
-        <mass
-          value="0.025" />
-      </inertial>
+          xyz="5.96744875736022E-16 -1.24475083018716E-14 -0.0215899999999933"
+          rpy="0 0 0" />
+        <mass
+          value="0.00499543658848208" />
+        <inertia
+          ixx="8.99919949242919E-07"
+          ixy="3.97046694025453E-23"
+          ixz="9.81863387100444E-22"
+          iyy="8.9991994924288E-07"
+          iyz="-8.0163727523739E-19"
+          izz="3.31951561004127E-07" />
+    </inertial>
       <visual>
         <origin
@@ -600,9 +698,16 @@
       <inertial>
         <origin
-          xyz="5.68989300120393E-16 -3.40699690681845E-15 -0.0215899999999933"
-          rpy="0 0 0" />
-        <mass
-          value="0.025" />
-      </inertial>
+          xyz="5.96744875736022E-16 -1.24475083018716E-14 -0.0215899999999933"
+          rpy="0 0 0" />
+        <mass
+          value="0.00499543658848208" />
+        <inertia
+          ixx="8.99919949242919E-07"
+          ixy="3.97046694025453E-23"
+          ixz="9.81863387100444E-22"
+          iyy="8.9991994924288E-07"
+          iyz="-8.0163727523739E-19"
+          izz="3.31951561004127E-07" />
+    </inertial>
       <visual>
         <origin
@@ -647,9 +752,16 @@
       <inertial>
         <origin
-          xyz="5.96744875736022E-16 -9.87751547221194E-15 -0.0215899999999933"
-          rpy="0 0 0" />
-        <mass
-          value="0.025" />
-      </inertial>
+          xyz="5.96744875736022E-16 -1.24475083018716E-14 -0.0215899999999933"
+          rpy="0 0 0" />
+        <mass
+          value="0.00499543658848208" />
+        <inertia
+          ixx="8.99919949242919E-07"
+          ixy="3.97046694025453E-23"
+          ixz="9.81863387100444E-22"
+          iyy="8.9991994924288E-07"
+          iyz="-8.0163727523739E-19"
+          izz="3.31951561004127E-07" />
+    </inertial>
       <visual>
         <origin
@@ -694,9 +806,16 @@
       <inertial>
         <origin
-          xyz="6.10622663543836E-16 -6.50608039665102E-15 -0.0215899999999933"
-          rpy="0 0 0" />
-        <mass
-          value="0.025" />
-      </inertial>
+          xyz="5.96744875736022E-16 -1.24475083018716E-14 -0.0215899999999933"
+          rpy="0 0 0" />
+        <mass
+          value="0.00499543658848208" />
+        <inertia
+          ixx="8.99919949242919E-07"
+          ixy="3.97046694025453E-23"
+          ixz="9.81863387100444E-22"
+          iyy="8.9991994924288E-07"
+          iyz="-8.0163727523739E-19"
+          izz="3.31951561004127E-07" />
+    </inertial>
       <visual>
         <origin
@@ -741,9 +860,16 @@
       <inertial>
         <origin
-          xyz="5.96744875736022E-16 -3.365797224264E-15 -0.0215899999999933"
-          rpy="0 0 0" />
-        <mass
-          value="0.025" />
-      </inertial>
+          xyz="5.96744875736022E-16 -1.24475083018716E-14 -0.0215899999999933"
+          rpy="0 0 0" />
+        <mass
+          value="0.00499543658848208" />
+        <inertia
+          ixx="8.99919949242919E-07"
+          ixy="3.97046694025453E-23"
+          ixz="9.81863387100444E-22"
+          iyy="8.9991994924288E-07"
+          iyz="-8.0163727523739E-19"
+          izz="3.31951561004127E-07" />
+    </inertial>
       <visual>
         <origin
@@ -788,9 +914,16 @@
       <inertial>
         <origin
-          xyz="5.82867087928207E-16 -3.35452152167015E-15 -0.0215899999999933"
-          rpy="0 0 0" />
-        <mass
-          value="0.025" />
-      </inertial>
+          xyz="5.96744875736022E-16 -1.24475083018716E-14 -0.0215899999999933"
+          rpy="0 0 0" />
+        <mass
+          value="0.00499543658848208" />
+        <inertia
+          ixx="8.99919949242919E-07"
+          ixy="3.97046694025453E-23"
+          ixz="9.81863387100444E-22"
+          iyy="8.9991994924288E-07"
+          iyz="-8.0163727523739E-19"
+          izz="3.31951561004127E-07" />
+    </inertial>
       <visual>
         <origin
