Commit message: Added inertia tags back to robot links so that robot can be used in gazebo

File: linorobot2_description/urdf/mech/mecanum_wheel_right.urdf.xacro (robot description, xacro)
@@ -5,8 +5,15 @@
       <inertial>
         <origin
-          xyz="-1.48571881243385E-15 -6.7886631592007E-16 -0.0136209233699844"
-          rpy="0 0 0" />
-        <mass
-          value="0.25" />
+        xyz="-1.48571881243385E-15 -6.7886631592007E-16 -0.0136209233699844"
+        rpy="0 0 0" />
+      <mass
+        value="0.0396439871820506" />
+      <inertia
+        ixx="3.76805204137311E-05"
+        ixy="1.66580607308995E-20"
+        ixz="3.71031510257902E-18"
+        iyy="3.76805204137311E-05"
+        iyz="1.63812405352096E-18"
+        izz="7.1054120055567E-05" />
       </inertial>
       <visual>
@@ -43,10 +50,17 @@
       name="${end}_${side}_drum">
       <inertial>
-        <origin
-          xyz="0.0136209233699844 6.56957443528167E-16 -1.48512976903392E-15"
-          rpy="0 0 0" />
-        <mass
-          value="0.5" />
-      </inertial>
+      <origin
+        xyz="0.0136209233699844 6.56957443528167E-16 -1.48512976903392E-15"
+        rpy="0 0 0" />
+      <mass
+        value="0.0396439871820506" />
+      <inertia
+        ixx="7.1054120055567E-05"
+        ixy="1.62690471844664E-18"
+        ixz="-3.70636817664487E-18"
+        iyy="3.76805204137311E-05"
+        iyz="1.0973915143622E-20"
+        izz="3.76805204137311E-05" />
+    </inertial>
       <visual>
         <origin
@@ -89,6 +103,17 @@
       name="${end}_${side}_plate1">
       <inertial>
-        <mass value="0.5" />
-      </inertial>
+      <origin
+        xyz="-0.00283756867072453 8.89413056967719E-16 2.68096171575045E-15"
+        rpy="0 0 0" />
+      <mass
+        value="0.0253986639693881" />
+      <inertia
+        ixx="8.39719993847471E-05"
+        ixy="1.90079838330856E-18"
+        ixz="4.7133202434868E-18"
+        iyy="4.21627753206921E-05"
+        iyz="-1.48230765769502E-20"
+        izz="4.21627753206921E-05" />
+    </inertial>
       <visual>
         <origin
@@ -131,6 +156,17 @@
       name="${end}_${side}_plate2">
       <inertial>
-        <mass value="0.5" />
-      </inertial>
+      <origin
+        xyz="-0.00283756867072453 -9.8249688244021E-17 5.89771118826868E-17"
+        rpy="0 0 0" />
+      <mass
+        value="0.0253986639693881" />
+      <inertia
+        ixx="8.39719993847471E-05"
+        ixy="-9.13983660820293E-21"
+        ixz="5.31128745957199E-22"
+        iyy="4.2162775320692E-05"
+        iyz="1.59877468794249E-20"
+        izz="4.21627753206921E-05" />
+    </inertial>
       <visual>
         <origin
@@ -173,10 +209,17 @@
       name="${end}_${side}_roller1">
       <inertial>
-        <origin
-          xyz="5.82867087928207E-16 3.51108031537706E-15 -0.0215899999999933"
-          rpy="0 0 0" />
-        <mass
-          value="0.025" />
-      </inertial>
+      <origin
+        xyz="5.82867087928207E-16 3.51108031537706E-15 -0.0215899999999933"
+        rpy="0 0 0" />
+      <mass
+        value="0.00499543658848254" />
+      <inertia
+        ixx="8.99919949255961E-07"
+        ixy="0"
+        ixz="7.14684049245816E-22"
+        iyy="8.999199492559E-07"
+        iyz="-8.01670362461892E-19"
+        izz="3.31951561028667E-07" />
+    </inertial>
       <visual>
         <origin
@@ -220,10 +263,17 @@
       name="${end}_${side}_roller2">
       <inertial>
-        <origin
-          xyz="5.68989300120393E-16 -1.90819582357449E-15 -0.0215899999999933"
-          rpy="0 0 0" />
-        <mass
-          value="0.025" />
-      </inertial>
+      <origin
+        xyz="5.82867087928207E-16 3.51108031537706E-15 -0.0215899999999933"
+        rpy="0 0 0" />
+      <mass
+        value="0.00499543658848254" />
+      <inertia
+        ixx="8.99919949255961E-07"
+        ixy="0"
+        ixz="7.14684049245816E-22"
+        iyy="8.999199492559E-07"
+        iyz="-8.01670362461892E-19"
+        izz="3.31951561028667E-07" />
+    </inertial>
       <visual>
         <origin
@@ -267,10 +317,17 @@
       name="${end}_${side}_roller3">
       <inertial>
-        <origin
-          xyz="5.82867087928207E-16 -4.16333634234434E-17 -0.0215899999999933"
-          rpy="0 0 0" />
-        <mass
-          value="0.025" />
-      </inertial>
+      <origin
+        xyz="5.82867087928207E-16 3.51108031537706E-15 -0.0215899999999933"
+        rpy="0 0 0" />
+      <mass
+        value="0.00499543658848254" />
+      <inertia
+        ixx="8.99919949255961E-07"
+        ixy="0"
+        ixz="7.14684049245816E-22"
+        iyy="8.999199492559E-07"
+        iyz="-8.01670362461892E-19"
+        izz="3.31951561028667E-07" />
+    </inertial>
       <visual>
         <origin
@@ -314,10 +371,17 @@
       name="${end}_${side}_roller4">
       <inertial>
-        <origin
-          xyz="5.89805981832114E-16 -3.20576898360514E-15 -0.0215899999999933"
-          rpy="0 0 0" />
-        <mass
-          value="0.025" />
-      </inertial>
+      <origin
+        xyz="5.82867087928207E-16 3.51108031537706E-15 -0.0215899999999933"
+        rpy="0 0 0" />
+      <mass
+        value="0.00499543658848254" />
+      <inertia
+        ixx="8.99919949255961E-07"
+        ixy="0"
+        ixz="7.14684049245816E-22"
+        iyy="8.999199492559E-07"
+        iyz="-8.01670362461892E-19"
+        izz="3.31951561028667E-07" />
+    </inertial>
       <visual>
         <origin
@@ -361,10 +425,17 @@
       name="${end}_${side}_roller5">
       <inertial>
-        <origin
-          xyz="5.82867087928207E-16 -7.39686090156511E-15 -0.0215899999999933"
-          rpy="0 0 0" />
-        <mass
-          value="0.025" />
-      </inertial>
+      <origin
+        xyz="5.82867087928207E-16 3.51108031537706E-15 -0.0215899999999933"
+        rpy="0 0 0" />
+      <mass
+        value="0.00499543658848254" />
+      <inertia
+        ixx="8.99919949255961E-07"
+        ixy="0"
+        ixz="7.14684049245816E-22"
+        iyy="8.999199492559E-07"
+        iyz="-8.01670362461892E-19"
+        izz="3.31951561028667E-07" />
+    </inertial>
       <visual>
         <origin
@@ -408,10 +479,17 @@
       name="${end}_${side}_roller6">
       <inertial>
-        <origin
-          xyz="5.89805981832114E-16 -9.20097331658098E-15 -0.0215899999999933"
-          rpy="0 0 0" />
-        <mass
-          value="0.025" />
-      </inertial>
+      <origin
+        xyz="5.82867087928207E-16 3.51108031537706E-15 -0.0215899999999933"
+        rpy="0 0 0" />
+      <mass
+        value="0.00499543658848254" />
+      <inertia
+        ixx="8.99919949255961E-07"
+        ixy="0"
+        ixz="7.14684049245816E-22"
+        iyy="8.999199492559E-07"
+        iyz="-8.01670362461892E-19"
+        izz="3.31951561028667E-07" />
+    </inertial>
       <visual>
         <origin
@@ -455,10 +533,17 @@
       name="${end}_${side}_roller7">
       <inertial>
-        <origin
-          xyz="5.89805981832114E-16 -8.25034485174569E-15 -0.0215899999999933"
-          rpy="0 0 0" />
-        <mass
-          value="0.025" />
-      </inertial>
+      <origin
+        xyz="5.82867087928207E-16 3.51108031537706E-15 -0.0215899999999933"
+        rpy="0 0 0" />
+      <mass
+        value="0.00499543658848254" />
+      <inertia
+        ixx="8.99919949255961E-07"
+        ixy="0"
+        ixz="7.14684049245816E-22"
+        iyy="8.999199492559E-07"
+        iyz="-8.01670362461892E-19"
+        izz="3.31951561028667E-07" />
+    </inertial>
       <visual>
         <origin
@@ -502,10 +587,17 @@
       name="${end}_${side}_roller8">
       <inertial>
-        <origin
-          xyz="5.759281940243E-16 2.22044604925031E-15 -0.0215899999999933"
-          rpy="0 0 0" />
-        <mass
-          value="0.025" />
-      </inertial>
+      <origin
+        xyz="5.82867087928207E-16 3.51108031537706E-15 -0.0215899999999933"
+        rpy="0 0 0" />
+      <mass
+        value="0.00499543658848254" />
+      <inertia
+        ixx="8.99919949255961E-07"
+        ixy="0"
+        ixz="7.14684049245816E-22"
+        iyy="8.999199492559E-07"
+        iyz="-8.01670362461892E-19"
+        izz="3.31951561028667E-07" />
+    </inertial>
       <visual>
         <origin
@@ -549,10 +641,17 @@
       name="${end}_${side}_roller9">
       <inertial>
-        <origin
-          xyz="5.759281940243E-16 -2.60208521396521E-15 -0.0215899999999933"
-          rpy="0 0 0" />
-        <mass
-          value="0.025" />
-      </inertial>
+      <origin
+        xyz="5.82867087928207E-16 3.51108031537706E-15 -0.0215899999999933"
+        rpy="0 0 0" />
+      <mass
+        value="0.00499543658848254" />
+      <inertia
+        ixx="8.99919949255961E-07"
+        ixy="0"
+        ixz="7.14684049245816E-22"
+        iyy="8.999199492559E-07"
+        iyz="-8.01670362461892E-19"
+        izz="3.31951561028667E-07" />
+    </inertial>
       <visual>
         <origin
@@ -596,10 +695,17 @@
       name="${end}_${side}_roller10">
       <inertial>
-        <origin
-          xyz="5.89805981832114E-16 -3.42087469462626E-15 -0.0215899999999933"
-          rpy="0 0 0" />
-        <mass
-          value="0.025" />
-      </inertial>
+      <origin
+        xyz="5.82867087928207E-16 3.51108031537706E-15 -0.0215899999999933"
+        rpy="0 0 0" />
+      <mass
+        value="0.00499543658848254" />
+      <inertia
+        ixx="8.99919949255961E-07"
+        ixy="0"
+        ixz="7.14684049245816E-22"
+        iyy="8.999199492559E-07"
+        iyz="-8.01670362461892E-19"
+        izz="3.31951561028667E-07" />
+    </inertial>
       <visual>
         <origin
@@ -643,10 +749,17 @@
       name="${end}_${side}_roller11">
       <inertial>
-        <origin
-          xyz="5.89805981832114E-16 -5.03069808033274E-15 -0.0215899999999933"
-          rpy="0 0 0" />
-        <mass
-          value="0.025" />
-      </inertial>
+      <origin
+        xyz="5.82867087928207E-16 3.51108031537706E-15 -0.0215899999999933"
+        rpy="0 0 0" />
+      <mass
+        value="0.00499543658848254" />
+      <inertia
+        ixx="8.99919949255961E-07"
+        ixy="0"
+        ixz="7.14684049245816E-22"
+        iyy="8.999199492559E-07"
+        iyz="-8.01670362461892E-19"
+        izz="3.31951561028667E-07" />
+    </inertial>
       <visual>
         <origin
@@ -690,10 +803,17 @@
       name="${end}_${side}_roller12">
       <inertial>
-        <origin
-          xyz="5.759281940243E-16 -3.44169137633799E-15 -0.0215899999999933"
-          rpy="0 0 0" />
-        <mass
-          value="0.025" />
-      </inertial>
+      <origin
+        xyz="5.82867087928207E-16 3.51108031537706E-15 -0.0215899999999933"
+        rpy="0 0 0" />
+      <mass
+        value="0.00499543658848254" />
+      <inertia
+        ixx="8.99919949255961E-07"
+        ixy="0"
+        ixz="7.14684049245816E-22"
+        iyy="8.999199492559E-07"
+        iyz="-8.01670362461892E-19"
+        izz="3.31951561028667E-07" />
+    </inertial>
       <visual>
         <origin
@@ -737,10 +857,17 @@
       name="${end}_${side}_roller13">
       <inertial>
-        <origin
-          xyz="5.89805981832114E-16 -3.36536354339501E-15 -0.0215899999999933"
-          rpy="0 0 0" />
-        <mass
-          value="0.025" />
-      </inertial>
+      <origin
+        xyz="5.82867087928207E-16 3.51108031537706E-15 -0.0215899999999933"
+        rpy="0 0 0" />
+      <mass
+        value="0.00499543658848254" />
+      <inertia
+        ixx="8.99919949255961E-07"
+        ixy="0"
+        ixz="7.14684049245816E-22"
+        iyy="8.999199492559E-07"
+        iyz="-8.01670362461892E-19"
+        izz="3.31951561028667E-07" />
+    </inertial>
       <visual>
         <origin
@@ -784,10 +911,17 @@
       name="${end}_${side}_roller14">
       <inertial>
-        <origin
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
File: linorobot2_description/urdf/mech/side_channel.urdf.xacro (robot description, xacro)
@@ -18,4 +18,11 @@
       <inertial>
         <mass value="5"/>
+        <inertia
+        ixx ="0.0027"
+        iyy ="0.2831"
+        izz ="0.2808"
+        ixy ="0.0"
+        ixz ="0.0"
+        iyz ="0.0"/>
       </inertial>
     </link>

File: linorobot2_description/urdf/robots/mecanum.urdf.xacro (robot description, xacro)
@@ -5,8 +5,8 @@
   <xacro:include filename="$(find linorobot2_description)/urdf/mech/mecanum_wheel_left.urdf.xacro" />
   <xacro:include filename="$(find linorobot2_description)/urdf/mech/mecanum_wheel_right.urdf.xacro" />
-  <xacro:include filename="$(find linorobot2_description)/urdf/sensors/imu.urdf.xacro" />
-  <xacro:include filename="$(find linorobot2_description)/urdf/sensors/generic_laser.urdf.xacro" />
-  <xacro:include filename="$(find linorobot2_description)/urdf/sensors/depth_sensor.urdf.xacro" />
-  <xacro:include filename="$(find linorobot2_description)/urdf/controllers/omni_drive.urdf.xacro" />
+  <!-- <xacro:include filename="$(find linorobot2_description)/urdf/sensors/imu.urdf.xacro" /> -->
+  <!-- <xacro:include filename="$(find linorobot2_description)/urdf/sensors/generic_laser.urdf.xacro" /> -->
+  <!-- <xacro:include filename="$(find linorobot2_description)/urdf/sensors/depth_sensor.urdf.xacro" /> -->
+  <!-- <xacro:include filename="$(find linorobot2_description)/urdf/controllers/omni_drive.urdf.xacro" /> -->
   <xacro:include filename="$(find linorobot2_description)/urdf/mech/end_channel.urdf.xacro" />
   <xacro:include filename="$(find linorobot2_description)/urdf/mech/side_channel.urdf.xacro" />
@@ -85,18 +85,7 @@
     <child link="front_rs_depth_optical_frame" />
   </joint>
+  <link name="front_rs_depth_optical_frame">
+  </link>
   <link name="rear_rs_depth_optical_frame">
-    <inertial>
-      <mass value="0.025" />
-    </inertial>
-    <visual>
-      <origin
-        xyz="0 0 0"
-        rpy="0 0 0" />
-    </visual>
-    <collision>
-      <origin
-        xyz="0 0 0"
-        rpy="0 0 0" />
-    </collision>
   </link>
   <!-- IsaacSim will likely not respect joint angles for realsense joints -->
@@ -110,17 +99,4 @@
   </joint>
   <link name="left_rs_depth_optical_frame">
-    <inertial>
-      <mass value="0.025" />
-    </inertial>
-    <visual>
-      <origin
-        xyz="0 0 0"
-        rpy="0 0 0" />
-    </visual>
-    <collision>
-      <origin
-        xyz="0 0 0"
-        rpy="0 0 0" />
-    </collision>
   </link>
   <!-- IsaacSim will likely not respect joint angles for realsense joints -->
@@ -134,17 +110,4 @@
   </joint>
   <link name="right_rs_depth_optical_frame">
-    <inertial>
-      <mass value="0.025" />
-    </inertial>
-    <visual>
-      <origin
-        xyz="0 0 0"
-        rpy="0 0 0" />
-    </visual>
-    <collision>
-      <origin
-        xyz="0 0 0"
-        rpy="0 0 0" />
-    </collision>
   </link>
   <!-- IsaacSim will likely not respect joint angles for realsense joints -->

Commit message: Front pcl properly transformed to base link now, cirumventing the transformation by the gazebo camera because it is incorrect

File: linorobot2_description/urdf/mech/base.urdf.xacro (robot description, xacro)
@@ -2,5 +2,5 @@
 <robot xmlns:xacro="http://ros.org/wiki/xacro">
   <xacro:macro name="base" params="length width height mass wheel_radius wheel_pos_z">
-    <link name="base_footprint"/>
+    <link name="base_footprint2"/>
     <link name="base_link">
       <visual>
@@ -9,7 +9,4 @@
           <box size="${length} ${width} ${height}"/>
         </geometry>
-        <material name="gray_base">
-          <color rgba="0.8 0.8 0.83 1.0"/>
-        </material>
       </visual>
       <collision>
@@ -25,16 +22,6 @@
       </inertial>
     </link>
-    <gazebo reference="base_link">
-      <visual>
-        <material>
-          <ambient>0.8392 0.6314 0.0 1.0</ambient>
-          <diffuse>0.8392 0.6314 0.0 1.0</diffuse>
-          <specular>0.99 0.99 0.99 1.0</specular>
-          <emissive>0.0 0.0 0.0 0.0</emissive>
-        </material>
-      </visual>
-    </gazebo>
     <joint name="base_to_footprint" type="fixed">
-      <parent link="base_footprint"/>
+      <parent link="base_footprint2"/>
       <child link="base_link"/>
       <origin xyz="0 0 ${wheel_radius - wheel_pos_z}" rpy="0 0 0"/>

File: linorobot2_description/urdf/mech/side_channel.urdf.xacro (robot description, xacro)
@@ -1,4 +1,4 @@
 <?xml version="1.0"?>
-<robot name="linorobot2_mecanum" xmlns:xacro="http://ros.org/wiki/xacro">
+<robot xmlns:xacro="http://ros.org/wiki/xacro">
   <xacro:macro name="side_channel" params="side pos_y">
     <link name="${side}_channel">

File: linorobot2_description/urdf/robots/camera.urdf.xacro (robot description, xacro)
@@ -28,5 +28,5 @@
           <imageTopicName>image_raw</imageTopicName>
           <cameraInfoTopicName>camera_info</cameraInfoTopicName>
-          <frameName>right_rs_depth_optical_frame</frameName>
+          <frameName>/front_rs_gazebo_camera_frame</frameName>
           <hackBaseline>0.07</hackBaseline>
           <distortionK1>0.0</distortionK1>
@@ -51,11 +51,10 @@
     <link name="${camera_pos}_gazebo_camera_frame">
     </link>
-    <!-- Gazebo camera has different frame than realsense camera, need a transform to get from realsense to gazebo camera -->
     <joint
-      name="${camera_pos}_rs_depth_optical_frame_to_${camera_pos}_gazebo_camera_frame" type="fixed">
+      name="base_link_to_${camera_pos}_gazebo_camera_frame" type="fixed">
       <origin
-        xyz="0 0 0"
-        rpy="1.57 -1.57 0" />
-      <parent link="${camera_pos}_rs_depth_optical_frame" />
+        xyz="0.3 0 0"
+        rpy="0 0 0" />
+      <parent link="base_link" />
       <child link="${camera_pos}_gazebo_camera_frame" />
     </joint>

File: linorobot2_description/urdf/robots/mecanum_libplanar.urdf.xacro (robot description, xacro)
@@ -1,4 +1,4 @@
 <?xml version="1.0"?>
-<robot name="linorobot2_mecanum" xmlns:xacro="http://ros.org/wiki/xacro">
+<robot name="linorobot2" xmlns:xacro="http://ros.org/wiki/xacro">
   <xacro:include filename="$(find linorobot2_description)/urdf/mecanum_properties.urdf.xacro" />
   <xacro:include filename="$(find linorobot2_description)/urdf/mech/base.urdf.xacro" />
@@ -8,13 +8,16 @@
   <xacro:include filename="$(find linorobot2_description)/urdf/mech/side_channel.urdf.xacro" />
   <xacro:include filename="$(find linorobot2_description)/urdf/robots/camera.urdf.xacro" />
-  <xacro:camera camera_pos="front" x="0.410335" y="0" z="0.0892"
-                                   r_rs="-1.57" p_rs="0" yaw_rs="-1.57" />
-  <xacro:camera camera_pos="left" x="0.0" y="0.247" z="0.089"
+  <!-- 0.0892 -->
+  <link name="base_link">
+  </link>
+  <xacro:camera camera_pos="front" x="0.410335" y="0" z="0.3"
+                                   r_rs= "-1.57" p_rs="0" yaw_rs="-1.57" />
+  <!-- <xacro:camera camera_pos="left" x="0.0" y="0.247" z="0.089"
                                   r_rs="-1.57" p_rs="0.0" yaw_rs="0"/>
   <xacro:camera camera_pos="rear" x="-0.41" y="0.0" z="0.089"
                                   r_rs="-1.57" p_rs="0" yaw_rs="1.57" />
   <xacro:camera camera_pos="right" x="0" y="-0.247" z="0.089"
-                                  r_rs="-1.57" p_rs="0" yaw_rs="3.14"/>
-  <gazebo>
+                                  r_rs="-1.57" p_rs="0" yaw_rs="3.14"/> -->
+  <!-- <gazebo>
     <plugin name="mecanum_wheel_mimic" filename="libgazebo_ros_planar_move.so">
       <ros>
@@ -29,6 +32,6 @@
       <publish_odom_tf>true</publish_odom_tf>
     </plugin>
-  </gazebo>
-  <xacro:base
+  </gazebo> -->
+  <!-- <xacro:base
     length="${base_length}"
     width="${base_width}"
@@ -37,6 +40,6 @@
     wheel_radius="${wheel_radius}"
     wheel_pos_z="${wheel_pos_z}"
-  />
-  <xacro:end_channel
+  /> -->
+  <!-- <xacro:end_channel
     end="front"
     pos_x="0.383345"
@@ -45,5 +48,5 @@
     end="back"
     pos_x="-0.383345"
-  />
+  /> -->
   <xacro:side_channel
     side="left"
