Commit message: Added a velocity scaler so that gazebo's planar movement speed is what we actually want. Need to add an odometry scalar to scale down the odometry coming out of the planar plugin

File: linorobot2_description/urdf/mech/base.urdf.xacro (robot description, xacro)
@@ -1,5 +1,5 @@
 <?xml version="1.0"?>
 <robot xmlns:xacro="http://ros.org/wiki/xacro">
-  <xacro:macro name="base" params="length width height mass">
+  <xacro:macro name="base" params="length width height">
     <link name="base_link">
       <visual>
@@ -14,9 +14,17 @@
           <box size="${length} ${width} ${height}"/>
         </geometry>
+        <surface>
+          <friction>
+            <ode>
+              <mu>0.0</mu>
+              <mu2>0.0</mu2>
+            </ode>
+          </friction>
+        </surface>
       </collision>
       <inertial>
         <origin xyz="0 0 0" rpy="0 0 0"/>
-        <mass value="${mass}"/>
-        <inertia ixx="0"  ixy="0"  ixz="0" iyy="0" iyz="0" izz="0" />
+        <mass value="0.01"/>
+        <inertia ixx="0.0004434"  ixy="0.000"  ixz="0.000" iyy="0.001785" iyz="0.000" izz="0.002179" />
       </inertial>
     </link>

File: linorobot2_description/urdf/mech/end_channel.urdf.xacro (robot description, xacro)
@@ -18,12 +18,12 @@
       <inertial>
         <origin xyz="0 0 0" rpy="0 0 0" />
-        <mass value="5"/>
+        <mass value="0.00"/>
         <inertia
-          ixx="0.1052"
+          ixx="0.0"
           ixy="0"
           ixz="0"
-          iyy="0.0042"
+          iyy="0.00"
           iyz="0"
-          izz="0.1034" />
+          izz="0.0" />
       </inertial>
     </link>

File: linorobot2_description/urdf/mech/mecanum_wheel_left_fixed.urdf.xacro (robot description, xacro)
@@ -6,12 +6,12 @@
       <inertial>
         <origin xyz="0 0 0" rpy="0 0 0"/>
-        <mass value="2.0"/>
+        <mass value="1.0"/>
         <inertia
-          ixx="0.000526666667"
+          ixx="0.00015"
           ixy="0"
           ixz="0"
-          iyy="0.000526666667"
+          iyy="0.00015"
           iyz="0"
-          izz="0.001"/>
+          izz="0.00025"/>
       </inertial>
       <visual>
@@ -27,10 +27,20 @@
           <cylinder radius="0.07162" length="0.05"/>
         </geometry>
+        <surface>
+          <friction>
+            <ode>
+              <mu>10000000.0</mu>
+              <mu2>10000000.0</mu2>
+            </ode>
+          </friction>
+        </surface>
       </collision>
     </link>
-    <joint name="base_link_to_${end}_${side}_wheel" type="fixed">
+    <joint name="base_link_to_${end}_${side}_wheel" type="continuous">
       <origin xyz="${pos_x} ${pos_y} 0"  rpy="1.57 0 0" />
       <parent link="base_link" />
       <child link="${end}_${side}_wheel" />
+      <axis xyz="0 0 1"/>
+      <dynamics damping="0.0" friction="0.1"/>
     </joint>
   </xacro:macro>

File: linorobot2_description/urdf/mech/side_channel.urdf.xacro (robot description, xacro)
@@ -17,9 +17,9 @@
       </collision>
       <inertial>
-        <mass value="5"/>
+        <mass value="0.00"/>
         <inertia
-        ixx ="0.0027"
-        iyy ="0.2831"
-        izz ="0.2808"
+        ixx ="0.00"
+        iyy ="0"
+        izz ="0"
         ixy ="0.0"
         ixz ="0.0"

File: linorobot2_description/urdf/robots/mecanum_libplanar.urdf.xacro (robot description, xacro)
@@ -27,8 +27,9 @@
     <plugin name="mecanum_wheel_mimic" filename="libgazebo_ros_planar_move.so">
       <ros>
-        <remapping>odom:=odom/unfiltered</remapping>
+        <remapping>odom:=/odom_unscaled</remapping>
+        <remapping>cmd_vel:=/cmd_vel_scaled</remapping>
       </ros>
       <command_topic>cmd_vel</command_topic>
-      <odometry_topic>odom/unfiltered</odometry_topic>
+      <odometry_topic>odom</odometry_topic>
       <odometry_frame>odom</odometry_frame>
       <odometry_rate>20.0</odometry_rate>
@@ -36,4 +37,6 @@
       <publish_odom>true</publish_odom>
       <publish_odom_tf>true</publish_odom_tf>
+      <update_rate>100</update_rate>
+      <publish_rate>10</publish_rate>
     </plugin>
   </gazebo>
@@ -42,7 +45,6 @@
     width="${base_width}"
     height="${base_height}"
-    mass="${base_mass}"
   />
-  <xacro:end_channel
+  <!-- <xacro:end_channel
     end="front"
     pos_x="0.383345"
@@ -59,6 +61,6 @@
     side="right"
     pos_y="-0.23653"
-  />
-  <xacro:mecanum_wheel_left
+  /> -->
+  <!-- <xacro:mecanum_wheel_left
     side="left"
     end="front"
@@ -83,4 +85,4 @@
     pos_x="${-wheel_pos_x}"
     pos_y="${-wheel_pos_y}"
-  />
+  /> -->
 </robot>
