Commit message: Cropping and downsampling pointclouds back in place

File: linorobot2_description/urdf/mech/base.urdf.xacro (robot description, xacro)
@@ -1,6 +1,5 @@
 <?xml version="1.0"?>
 <robot xmlns:xacro="http://ros.org/wiki/xacro">
-  <xacro:macro name="base" params="length width height mass wheel_radius wheel_pos_z">
-    <link name="base_footprint2"/>
+  <xacro:macro name="base" params="length width height mass">
     <link name="base_link">
       <visual>
@@ -18,13 +17,8 @@
       <inertial>
         <origin xyz="0 0 0" rpy="0 0 0"/>
-        <mass value="0"/>
+        <mass value="${mass}"/>
         <inertia ixx="0"  ixy="0"  ixz="0" iyy="0" iyz="0" izz="0" />
       </inertial>
     </link>
-    <joint name="base_to_footprint" type="fixed">
-      <parent link="base_footprint2"/>
-      <child link="base_link"/>
-      <origin xyz="0 0 ${wheel_radius - wheel_pos_z}" rpy="0 0 0"/>
-    </joint>
   </xacro:macro>
 </robot>

File: linorobot2_description/urdf/mech/mecanum_wheel_left_fixed.urdf.xacro (robot description, xacro)
@@ -5,43 +5,30 @@
     <link name="${end}_${side}_wheel">
       <inertial>
-        <origin
-          xyz="-3.9077136779291E-16 -0.0136205707454137 -1.44489682185117E-14"
-          rpy="0 0 0" />
-        <mass
-          value="0.039620820516108" />
+        <origin xyz="0 0 0" rpy="0 0 0"/>
+        <mass value="2.0"/>
         <inertia
-          ixx="3.76577202480009E-05"
-          ixy="-1.07908308681007E-19"
-          ixz="3.89356499633093E-22"
-          iyy="7.10123305553507E-05"
-          iyz="-1.66085499471637E-18"
-          izz="3.76577202480009E-05" />
+          ixx="0.000526666667"
+          ixy="0"
+          ixz="0"
+          iyy="0.000526666667"
+          iyz="0"
+          izz="0.001"/>
       </inertial>
       <visual>
-        <origin
-          xyz="0 0 0"
-          rpy="0 0 0" />
         <geometry>
-          <mesh
-            filename="package://linorobot2_description/mecanum_wheel_left/meshes/fixed_wheel.STL" />
+          <cylinder radius="0.07162" length="0.05"/>
         </geometry>
-        <material
-          name="">
-          <color
-            rgba="0.898039215686275 0.917647058823529 0.929411764705882 1" />
+        <material name="gray">
+          <color rgba="0.70 0.70 0.73 1.0"/>
         </material>
       </visual>
       <collision>
-        <origin
-          xyz="0 0 0"
-          rpy="0 0 0" />
         <geometry>
-          <mesh
-            filename="package://linorobot2_description/mecanum_wheel_left/meshes/fixed_wheel.STL" />
+          <cylinder radius="0.07162" length="0.05"/>
         </geometry>
       </collision>
     </link>
     <joint name="base_link_to_${end}_${side}_wheel" type="fixed">
-      <origin xyz="${pos_x} ${pos_y} 0"  rpy="0 0 0" />
+      <origin xyz="${pos_x} ${pos_y} 0"  rpy="1.57 0 0" />
       <parent link="base_link" />
       <child link="${end}_${side}_wheel" />

File: linorobot2_description/urdf/mech/mecanum_wheel_right_fixed.urdf.xacro (robot description, xacro)
@@ -4,38 +4,25 @@
     <link name="${end}_${side}_wheel">
       <inertial>
-        <origin
-        xyz="-1.48571881243385E-15 -6.7886631592007E-16 -0.0136209233699844"
-        rpy="0 0 0" />
-      <mass
-        value="0.0396439871820506" />
-      <inertia
-        ixx="3.76805204137311E-05"
-        ixy="1.66580607308995E-20"
-        ixz="3.71031510257902E-18"
-        iyy="3.76805204137311E-05"
-        iyz="1.63812405352096E-18"
-        izz="7.1054120055567E-05" />
+        <origin xyz="0 0 0" rpy="0 0 0"/>
+        <mass value="2.0"/>
+        <inertia
+          ixx="0.000526666667"
+          ixy="0"
+          ixz="0"
+          iyy="0.000526666667"
+          iyz="0"
+          izz="0.001"/>
       </inertial>
       <visual>
-        <origin
-          xyz="0 0 0"
-          rpy="0 0 0" />
         <geometry>
-          <mesh
-            filename="package://linorobot2_description/mecanum_wheel_right/meshes/fixed_wheel.STL" />
+          <cylinder radius="0.07162" length="0.05"/>
         </geometry>
-        <material
-          name="">
-          <color
-            rgba="0.898039215686275 0.917647058823529 0.929411764705882 1" />
+        <material name="gray">
+          <color rgba="0.70 0.70 0.73 1.0"/>
         </material>
       </visual>
       <collision>
-        <origin
-          xyz="0 0 0"
-          rpy="0 0 0" />
         <geometry>
-          <mesh
-            filename="package://linorobot2_description/mecanum_wheel_right/meshes/fixed_wheel.STL" />
+          <cylinder radius="0.07162" length="0.05"/>
         </geometry>
       </collision>

File: linorobot2_description/urdf/robots/mecanum_libplanar.urdf.xacro (robot description, xacro)
@@ -4,28 +4,25 @@
   <xacro:include filename="$(find linorobot2_description)/urdf/mech/base.urdf.xacro" />
   <xacro:include filename="$(find linorobot2_description)/urdf/mech/mecanum_wheel_left_fixed.urdf.xacro" />
-  <xacro:include filename="$(find linorobot2_description)/urdf/mech/mecanum_wheel_right_fixed.urdf.xacro" />
   <xacro:include filename="$(find linorobot2_description)/urdf/mech/end_channel.urdf.xacro" />
   <xacro:include filename="$(find linorobot2_description)/urdf/mech/side_channel.urdf.xacro" />
   <xacro:include filename="$(find linorobot2_description)/urdf/robots/camera.urdf.xacro" />
-  <!-- 0.0892 -->
-  <link name="base_link">
-  </link>
-  <xacro:camera camera_pos="front" x="0.410335" y="0" z="0.089"
+  <xacro:property name="rs_height" value="${base_height/2 + 0.05}" />
+  <xacro:camera camera_pos="front" x="0.410335" y="0" z="${rs_height}"
                                    r_rs= "-1.57" p_rs="0" yaw_rs="-1.57"
                                    r_cam="0" p_cam="0" yaw_cam="0"
                                    />
-  <xacro:camera camera_pos="left" x="0.0" y="0.247" z="0.089"
+  <xacro:camera camera_pos="left" x="0.0" y="0.247" z="${rs_height}"
                                   r_rs="-1.57" p_rs="0.0" yaw_rs="0"
                                   r_cam="0" p_cam="0" yaw_cam="1.57"
                                   />
-  <xacro:camera camera_pos="rear" x="-0.41" y="0.0" z="0.089"
+  <xacro:camera camera_pos="rear" x="-0.41" y="0.0" z="${rs_height}"
                                   r_rs="-1.57" p_rs="0" yaw_rs="1.57"
                                   r_cam="0" p_cam="0" yaw_cam="3.14"
                                   />
-  <xacro:camera camera_pos="right" x="0" y="-0.247" z="0.089"
+  <xacro:camera camera_pos="right" x="0" y="-0.247" z="${rs_height}"
                                   r_rs="-1.57" p_rs="0" yaw_rs="3.14"
                                   r_cam="0" p_cam="0" yaw_cam="-1.57"
                                   />
-  <!-- <gazebo>
+  <gazebo>
     <plugin name="mecanum_wheel_mimic" filename="libgazebo_ros_planar_move.so">
       <ros>
@@ -36,22 +33,20 @@
       <odometry_frame>odom</odometry_frame>
       <odometry_rate>20.0</odometry_rate>
-      <robot_base_frame>base_footprint</robot_base_frame>
+      <robot_base_frame>base_link</robot_base_frame>
       <publish_odom>true</publish_odom>
       <publish_odom_tf>true</publish_odom_tf>
     </plugin>
-  </gazebo> -->
-  <!-- <xacro:base
+  </gazebo>
+  <xacro:base
     length="${base_length}"
     width="${base_width}"
     height="${base_height}"
     mass="${base_mass}"
-    wheel_radius="${wheel_radius}"
-    wheel_pos_z="${wheel_pos_z}"
-  /> -->
-  <!-- <xacro:end_channel
+  />
+  <xacro:end_channel
     end="front"
     pos_x="0.383345"
   />
-  <xacro:end_channel
+  <!-- <xacro:end_channel
     end="back"
     pos_x="-0.383345"
@@ -65,5 +60,5 @@
     pos_y="-0.23653"
   />
-  <!-- <xacro:mecanum_wheel_left
+  <xacro:mecanum_wheel_left
     side="left"
     end="front"
@@ -71,5 +66,5 @@
     pos_y="${wheel_pos_y}"
   />
-  <xacro:mecanum_wheel_right
+  <xacro:mecanum_wheel_left
     side="right"
     end="front"
@@ -77,5 +72,5 @@
     pos_y="${-wheel_pos_y}"
   />
-  <xacro:mecanum_wheel_right
+  <xacro:mecanum_wheel_left
     side="left"
     end="rear"
@@ -88,4 +83,4 @@
     pos_x="${-wheel_pos_x}"
     pos_y="${-wheel_pos_y}"
-  /> -->
+  />
 </robot>

Commit message: Added namespacing to frames, since all frames get publsihed to tf topic

File: linorobot2_description/urdf/mech/base.urdf.xacro (robot description, xacro)
@@ -1,10 +1,10 @@
 <?xml version="1.0"?>
 <robot xmlns:xacro="http://ros.org/wiki/xacro">
-  <xacro:macro name="base" params="length width height">
+  <xacro:macro name="base" params="namespace length width height">
     <!-- Beware changing masses or inertias of the base link. It will affect the robot's motion. -->
     <!-- Gazebos planar move model moves the robot at a different velocity than requested, but publishes the requested velocity in odometry. -->
     <!-- A linear transformation between desired and actual velocity is applied to the velocity going into Gazebo planar movement, and to the odom coming out of Gazebo planar movement -->
     <!-- This linear transformation will change in the physics of the robot changes, so beware changing masses or inertias of the base link. -->
-    <link name="base_link">
+    <link name="${namespace}_base_link">
       <visual>
         <origin xyz="0 0 0" rpy="0 0 0"/>

File: linorobot2_description/urdf/robots/camera.urdf.xacro (robot description, xacro)
@@ -2,6 +2,6 @@
 <robot name="linorobot2_mecanum" xmlns:xacro="http://ros.org/wiki/xacro">
   <xacro:macro name="camera" params="namespace camera_pos x y z r_rs p_rs yaw_rs r_cam p_cam yaw_cam">
-    <gazebo reference="${camera_pos}_gazebo_camera_frame">
-    <sensor type="depth" name="${camera_pos}_camera">
+    <gazebo reference="${namespace}_${camera_pos}_gazebo_camera_frame">
+    <sensor type="depth" name="${namespace}_${camera_pos}_camera">
       <update_rate>15.0</update_rate>
       <camera>
@@ -22,5 +22,5 @@
         </noise>
       </camera>
-      <plugin name="${camera_pos}_camera_controller" filename="libgazebo_ros_camera.so">
+      <plugin name="${namespace}_${camera_pos}_camera_controller" filename="libgazebo_ros_camera.so">
         <ros>
             <namespace>${namespace}</namespace>
@@ -32,5 +32,5 @@
         <imageTopicName>image_raw</imageTopicName>
         <cameraInfoTopicName>camera_info</cameraInfoTopicName>
-        <frameName>/${camera_pos}_rs_gazebo_camera_frame</frameName>
+        <frameName>${namespace}_${camera_pos}_rs_gazebo_camera_frame</frameName>
         <hackBaseline>0.07</hackBaseline>
         <distortionK1>0.0</distortionK1>
@@ -42,23 +42,23 @@
     </sensor>
   </gazebo>
-    <link name="${camera_pos}_rs_depth_optical_frame">
+    <link name="${namespace}_${camera_pos}_rs_depth_optical_frame">
     </link>
     <joint
-      name="base_link_to_${camera_pos}_rs" type="fixed">
+      name="${namespace}_base_link_to_${camera_pos}_rs" type="fixed">
       <origin
         xyz="${x} ${y} ${z}"
         rpy="${r_rs} ${p_rs} ${yaw_rs}" />
-      <parent link="base_link" />
-      <child link="${camera_pos}_rs_depth_optical_frame" />
+      <parent link="${namespace}_base_link" />
+      <child link="${namespace}_${camera_pos}_rs_depth_optical_frame" />
     </joint>
-    <link name="${camera_pos}_gazebo_camera_frame">
+    <link name="${namespace}_${camera_pos}_gazebo_camera_frame">
     </link>
     <joint
-      name="base_link_to_${camera_pos}_gazebo_camera_frame" type="fixed">
+      name="${namespace}_base_link_to_${camera_pos}_gazebo_camera_frame" type="fixed">
       <origin
         xyz="${x} ${y} ${z}"
         rpy="${r_cam} ${p_cam} ${yaw_cam}" />
-      <parent link="base_link" />
-      <child link="${camera_pos}_gazebo_camera_frame" />
+      <parent link="${namespace}_base_link" />
+      <child link="${namespace}_${camera_pos}_gazebo_camera_frame" />
     </joint>
   </xacro:macro>

File: linorobot2_description/urdf/robots/mecanum_libplanar.urdf.xacro (robot description, xacro)
@@ -1,5 +1,5 @@
 <?xml version="1.0"?>
 <robot name="linorobot2" xmlns:xacro="http://www.ros.org/wiki/xacro">
-  <xacro:arg name="namespace" default="drone0"/>
+  <xacro:arg name="namespace" default=""/>
   <xacro:include filename="$(find linorobot2_description)/urdf/mecanum_properties.urdf.xacro" />
   <xacro:include filename="$(find linorobot2_description)/urdf/mech/base.urdf.xacro" />
@@ -32,12 +32,12 @@
       <ros>
         <namespace>$(arg namespace)</namespace>
-        <remapping>odom:=/odom_unscaled</remapping>
-        <remapping>cmd_vel:=/cmd_vel_scaled</remapping>
+        <remapping>odom:=odom_unscaled</remapping>
+        <remapping>cmd_vel:=cmd_vel_scaled</remapping>
       </ros>
       <command_topic>cmd_vel</command_topic>
       <odometry_topic>odom</odometry_topic>
-      <odometry_frame>odom</odometry_frame>
+      <odometry_frame>$(arg namespace)_odom</odometry_frame>
       <odometry_rate>20.0</odometry_rate>
-      <robot_base_frame>base_link</robot_base_frame>
+      <robot_base_frame>$(arg namespace)_base_link</robot_base_frame>
       <publish_odom>true</publish_odom>
       <publish_odom_tf>true</publish_odom_tf>
@@ -47,4 +47,5 @@
   </gazebo>
   <xacro:base
+    namespace="$(arg namespace)"
     length="${base_length}"
     width="${base_width}"

Commit message: got worker and drone connecting with gazebo plugin

File: linorobot2_description/urdf/mech/base.urdf.xacro (robot description, xacro)
@@ -18,19 +18,50 @@
           <box size="${length} ${width} ${height}"/>
         </geometry>
-        <surface>
-          <friction>
-            <ode>
-              <mu>0.0</mu>
-              <mu2>0.0</mu2>
-            </ode>
-          </friction>
-        </surface>
       </collision>
       <inertial>
         <origin xyz="0 0 0" rpy="0 0 0"/>
-        <mass value="0.01"/>
-        <inertia ixx="0.00009552"  ixy="0.000"  ixz="0.000" iyy="0.0003639" iyz="0.000" izz="0.0037" />
+        <mass value="20"/> <!-- Small, non-zero mass -->
+        <inertia
+          ixx="1.14"
+          ixy="-4.74983711945811E-18"
+          ixz="-1.80635263223563E-18"
+          iyy="1.53"
+          iyz="6.42624983676543E-18"
+          izz="0.43" />
       </inertial>
     </link>
+  <gazebo reference="${namespace}_base_link">
+    <material>Gazebo/White</material>
+    <turnGravityOff>false</turnGravityOff>
+    <selfCollide>true</selfCollide>
+    <mu1>0.0</mu1>
+    <mu2>0.0</mu2>
+  </gazebo>
+  <link name="${namespace}_attachment_point">
+      <inertial>
+        <origin xyz="0 0 0" rpy="0 0 0"/>
+        <mass value="0.01"/> <!-- Small, non-zero mass -->
+        <inertia
+          ixx="0.0001"
+          ixy="0"
+          ixz="0"
+          iyy="0.0001"
+          iyz="0"
+          izz="0.0001" />
+      </inertial>
+    </link>
+  <gazebo reference="${namespace}_attachment_point">
+    <material>Gazebo/Gray</material>
+    <turnGravityOff>false</turnGravityOff>
+    <selfCollide>true</selfCollide>
+  </gazebo>
+  <joint name="${namespace}_attachment_to_base" type="fixed">
+    <parent link="${namespace}_base_link"/>
+    <child link="${namespace}_attachment_point"/>
+    <origin xyz="0 0 0.6" rpy="0 0 1.57"/>
+  </joint>
+  <gazebo reference='${namespace}_attachment_to_base'>
+    <preserveFixedJoint>true</preserveFixedJoint>
+  </gazebo>
   </xacro:macro>
 </robot>

File: linorobot2_description/urdf/robots/mecanum_libplanar.urdf.xacro (robot description, xacro)
@@ -52,54 +52,3 @@
     height="${base_height}"
   />
-  <!-- Sliding platform link -->
-  <link name="$(arg namespace)_sliding_platform">
-    <visual>
-      <origin xyz="0 0 0" rpy="0 0 0"/>
-      <geometry>
-        <box size="${base_length} ${base_width} 0.05"/>
-      </geometry>
-      <material name="gray">
-        <color rgba="0.5 0.5 0.5 1"/>
-      </material>
-    </visual>
-    <collision>
-      <origin xyz="0 0 0" rpy="0 0 0"/>
-      <geometry>
-        <box size="${base_length} ${base_width} 0.05"/>
-      </geometry>
-    </collision>
-    <inertial>
-      <mass value="0.1"/> <!-- Small, non-zero mass -->
-      <inertia ixx="0.001" ixy="0.0" ixz="0.0" iyy="0.001" iyz="0.0" izz="0.001"/>
-    </inertial>
-  </link>
-  <!-- Prismatic joint for vertical sliding -->
-  <joint name="$(arg namespace)_sliding_joint" type="prismatic">
-    <parent link="$(arg namespace)_base_link"/>
-    <child link="$(arg namespace)_sliding_platform"/>
-    <origin xyz="0 0 ${base_height/2+0.05}" rpy="0 0 0"/>
-    <axis xyz="0 0 1"/>
-    <limit lower="0" upper="0.5" effort="100" velocity="0.5"/>
-  </joint>
-  <gazebo>
-    <plugin name="joint_state_publisher" filename="libgazebo_ros_joint_state_publisher.so">
-      <ros>
-        <namespace>$(arg namespace)</namespace>
-        <remapping>joint_states:=joint_states</remapping>
-      </ros>
-      <update_rate>30</update_rate>
-      <joint_name>$(arg namespace)_sliding_joint</joint_name>
-    </plugin>
-  </gazebo>
-  <gazebo>
-    <plugin name="gazebo_ros_joint_pose_trajectory"
-        filename="libgazebo_ros_joint_pose_trajectory.so">
-        <ros>
-          <!-- <namespace>$(arg namespace)</namespace> -->
-        </ros>
-        <update_rate>20</update_rate>
-        <frame_id>drone_boris_base_link</frame_id>
-        <!-- <joint_name>$(arg namespace)_sliding_joint</joint_name> -->
-    </plugin>
-  </gazebo>
 </robot>
