Commit message: All 4 wheels mounted to robot in gazebo, but rollers have no resistance, and robot glides around without any input

File: linorobot2_description/urdf/mecanum_properties.urdf.xacro (robot description, xacro)
@@ -1,5 +1,5 @@
 <?xml version="1.0"?>
 <robot xmlns:xacro="http://ros.org/wiki/xacro">
-  <xacro:property name="base_length" value="0.82067" />
+  <xacro:property name="base_length" value="0.65" />
   <xacro:property name="base_width" value="0.3175" />
   <xacro:property name="base_height" value="0.07772" />

File: linorobot2_description/urdf/mech/mecanum_wheel_left.urdf.xacro (robot description, xacro)
@@ -223,5 +223,5 @@
           iyz="-8.0163727523739E-19"
           izz="3.31951561004127E-07" />
-     </inertial>
+      </inertial>
       <visual>
         <origin
@@ -277,5 +277,5 @@
           iyz="-8.0163727523739E-19"
           izz="3.31951561004127E-07" />
-    </inertial>
+      </inertial>
       <visual>
         <origin
@@ -331,5 +331,5 @@
           iyz="-8.0163727523739E-19"
           izz="3.31951561004127E-07" />
-    </inertial>
+      </inertial>
       <visual>
         <origin
@@ -385,5 +385,5 @@
           iyz="-8.0163727523739E-19"
           izz="3.31951561004127E-07" />
-    </inertial>
+      </inertial>
       <visual>
         <origin
@@ -439,5 +439,5 @@
           iyz="-8.0163727523739E-19"
           izz="3.31951561004127E-07" />
-    </inertial>
+      </inertial>
       <visual>
         <origin
@@ -493,5 +493,5 @@
           iyz="-8.0163727523739E-19"
           izz="3.31951561004127E-07" />
-    </inertial>
+      </inertial>
       <visual>
         <origin
@@ -547,5 +547,5 @@
           iyz="-8.0163727523739E-19"
           izz="3.31951561004127E-07" />
-    </inertial>
+      </inertial>
       <visual>
         <origin
@@ -601,5 +601,5 @@
           iyz="-8.0163727523739E-19"
           izz="3.31951561004127E-07" />
-    </inertial>
+      </inertial>
       <visual>
         <origin
@@ -655,5 +655,5 @@
           iyz="-8.0163727523739E-19"
           izz="3.31951561004127E-07" />
-    </inertial>
+      </inertial>
       <visual>
         <origin
@@ -709,5 +709,5 @@
           iyz="-8.0163727523739E-19"
           izz="3.31951561004127E-07" />
-    </inertial>
+      </inertial>
       <visual>
         <origin
@@ -763,5 +763,5 @@
           iyz="-8.0163727523739E-19"
           izz="3.31951561004127E-07" />
-    </inertial>
+      </inertial>
       <visual>
         <origin
@@ -817,5 +817,5 @@
           iyz="-8.0163727523739E-19"
           izz="3.31951561004127E-07" />
-    </inertial>
+      </inertial>
       <visual>
         <origin
@@ -871,5 +871,5 @@
           iyz="-8.0163727523739E-19"
           izz="3.31951561004127E-07" />
-    </inertial>
+      </inertial>
       <visual>
         <origin
@@ -925,5 +925,5 @@
           iyz="-8.0163727523739E-19"
           izz="3.31951561004127E-07" />
-    </inertial>
+      </inertial>
       <visual>
         <origin

File: linorobot2_description/urdf/mech/mecanum_wheel_right.urdf.xacro (robot description, xacro)
@@ -258,5 +258,5 @@
       <axis
         xyz="0 0 1" />
-      <dynamics damping="0.1" friction="0.01"/>
+      <!--<dynamics damping="0.1" friction="0.01"/>-->
     </joint>
     <link
@@ -312,5 +312,5 @@
       <axis
         xyz="0 0 1" />
-      <dynamics damping="0.1" friction="0.01"/>
+      <!--<dynamics damping="0.1" friction="0.01"/>-->
     </joint>
     <link
@@ -366,5 +366,5 @@
       <axis
         xyz="0 0 1" />
-      <dynamics damping="0.1" friction="0.01"/>
+      <!--<dynamics damping="0.1" friction="0.01"/>-->
     </joint>
     <link
@@ -420,5 +420,5 @@
       <axis
         xyz="0 0 1" />
-      <dynamics damping="0.1" friction="0.01"/>
+      <!--<dynamics damping="0.1" friction="0.01"/>-->
     </joint>
     <link
@@ -474,5 +474,5 @@
       <axis
         xyz="0 0 1" />
-      <dynamics damping="0.1" friction="0.01"/>
+      <!--<dynamics damping="0.1" friction="0.01"/>-->
     </joint>
     <link
@@ -528,5 +528,5 @@
       <axis
         xyz="0 0 1" />
-      <dynamics damping="0.1" friction="0.01"/>
+      <!--<dynamics damping="0.1" friction="0.01"/>-->
     </joint>
     <link
@@ -582,5 +582,5 @@
       <axis
         xyz="0 0 1" />
-      <dynamics damping="0.1" friction="0.01"/>
+      <!--<dynamics damping="0.1" friction="0.01"/>-->
     </joint>
     <link
@@ -636,5 +636,5 @@
       <axis
         xyz="0 0 1" />
-      <dynamics damping="0.1" friction="0.01"/>
+      <!--<dynamics damping="0.1" friction="0.01"/>-->
     </joint>
     <link
@@ -690,5 +690,5 @@
       <axis
         xyz="0 0 1" />
-      <dynamics damping="0.1" friction="0.01"/>
+      <!--<dynamics damping="0.1" friction="0.01"/>-->
     </joint>
     <link
@@ -744,5 +744,5 @@
       <axis
         xyz="0 0 1" />
-      <dynamics damping="0.1" friction="0.01"/>
+      <!--<dynamics damping="0.1" friction="0.01"/>-->
     </joint>
     <link
@@ -798,5 +798,5 @@
       <axis
         xyz="0 0 1" />
-      <dynamics damping="0.1" friction="0.01"/>
+      <!--<dynamics damping="0.1" friction="0.01"/>-->
     </joint>
     <link
@@ -852,5 +852,5 @@
       <axis
         xyz="0 0 1" />
-      <dynamics damping="0.1" friction="0.01"/>
+      <!--<dynamics damping="0.1" friction="0.01"/>-->
     </joint>
     <link
@@ -906,5 +906,5 @@
       <axis
         xyz="0 0 1" />
-      <dynamics damping="0.1" friction="0.01"/>
+      <!--<dynamics damping="0.1" friction="0.01"/>-->
     </joint>
     <link
@@ -960,5 +960,5 @@
       <axis
         xyz="0 0 1" />
-      <dynamics damping="0.1" friction="0.01"/>
+      <!--<dynamics damping="0.1" friction="0.01"/>-->
     </joint>
     <link
@@ -1014,5 +1014,5 @@
       <axis
         xyz="0 0 1" />
-      <dynamics damping="0.1" friction="0.01"/>
+      <!--<dynamics damping="0.1" friction="0.01"/>-->
     </joint>
   </xacro:macro>

File: linorobot2_description/urdf/robots/mecanum.urdf.xacro (robot description, xacro)
@@ -45,5 +45,5 @@
     mass="${wheel_mass}"
   />
-  <!-- <xacro:mecanum_wheel_right
+  <xacro:mecanum_wheel_right
     side="right"
     end="front"
@@ -54,7 +54,7 @@
     pos_z="${wheel_pos_z}"
     mass="${wheel_mass}"
-  /> -->
+  />
   <!-- Back wheels mechanum style swapped (left mecanum wheel goes on right side of robot, and vice versa) -->
-  <!-- <xacro:mecanum_wheel_right
+  <xacro:mecanum_wheel_right
     side="left"
     end="rear"
@@ -75,5 +75,5 @@
     pos_z="${wheel_pos_z}"
     mass="${wheel_mass}"
-  /> -->
+  />
   <!-- IsaacSim will likely not respect joint angles for realsense joints -->
   <joint

Commit message: Corrected scaling for rotation, also found that increasing Izz in base link inertia made the robot move faster, oddly

File: linorobot2_description/urdf/mecanum_properties.urdf.xacro (robot description, xacro)
@@ -3,5 +3,5 @@
   <xacro:property name="base_length" value="0.65" />
   <xacro:property name="base_width" value="0.3175" />
-  <xacro:property name="base_height" value="0.07772" />
+  <xacro:property name="base_height" value="0.1189" />
   <xacro:property name="base_mass" value="30" />
   <xacro:property name="wheel_radius" value="0.07162" />

File: linorobot2_description/urdf/mech/base.urdf.xacro (robot description, xacro)
@@ -26,5 +26,5 @@
         <origin xyz="0 0 0" rpy="0 0 0"/>
         <mass value="0.01"/>
-        <inertia ixx="0.0004434"  ixy="0.000"  ixz="0.000" iyy="0.001785" iyz="0.000" izz="0.002179" />
+        <inertia ixx="0.00009552"  ixy="0.000"  ixz="0.000" iyy="0.0003639" iyz="0.000" izz="0.0037" />
       </inertial>
     </link>

Commit message: Got gazebo depth cam FOV setup properly to match realsense FOV

File: linorobot2_description/urdf/mecanum_properties.urdf.xacro (robot description, xacro)
@@ -1,7 +1,7 @@
 <?xml version="1.0"?>
 <robot xmlns:xacro="http://ros.org/wiki/xacro">
-  <xacro:property name="base_length" value="0.65" />
-  <xacro:property name="base_width" value="0.3175" />
-  <xacro:property name="base_height" value="0.1189" />
+  <xacro:property name="base_length" value="0.82" />
+  <xacro:property name="base_width" value="0.495" />
+  <xacro:property name="base_height" value="0.116" />
   <xacro:property name="base_mass" value="30" />
   <xacro:property name="wheel_radius" value="0.07162" />

File: linorobot2_description/urdf/robots/camera.urdf.xacro (robot description, xacro)
@@ -3,39 +3,40 @@
   <xacro:macro name="camera" params="camera_pos x y z r_rs p_rs yaw_rs r_cam p_cam yaw_cam">
     <gazebo reference="${camera_pos}_gazebo_camera_frame">
-      <sensor type="depth" name="${camera_pos}_camera">
-        <update_rate>15.0</update_rate>
-        <depth_camera name="${camera_pos}_camera">
-          <horizontal_fov>2.96</horizontal_fov>
-          <image>
-            <width>480</width>
-            <height>270</height>
-            <format>R8G8B8</format>
-          </image>
-          <clip>
-            <near>0.02</near>
-            <far>3</far>
-          </clip>
-          <noise>
-            <type>gaussian</type>
-            <mean>0.0</mean>
-            <stddev>0.007</stddev>
-          </noise>
-        </depth_camera>
-        <plugin name="${camera_pos}_camera_controller" filename="libgazebo_ros_camera.so">
-          <alwaysOn>true</alwaysOn>
-          <updateRate>0.0</updateRate>
-          <cameraName>${camera_pos}_camera</cameraName>
-          <imageTopicName>image_raw</imageTopicName>
-          <cameraInfoTopicName>camera_info</cameraInfoTopicName>
-          <frameName>/front_rs_gazebo_camera_frame</frameName>
-          <hackBaseline>0.07</hackBaseline>
-          <distortionK1>0.0</distortionK1>
-          <distortionK2>0.0</distortionK2>
-          <distortionK3>0.0</distortionK3>
-          <distortionT1>0.0</distortionT1>
-          <distortionT2>0.0</distortionT2>
-        </plugin>
-      </sensor>
-    </gazebo>
+    <sensor type="depth" name="${camera_pos}_camera">
+      <update_rate>15.0</update_rate>
+      <camera>
+        <horizontal_fov>1.5</horizontal_fov>
+        <image>
+          <width>480</width>
+          <height>270</height>
+          <format>R8G8B8</format>
+        </image>
+        <clip>
+          <near>0.02</near>
+          <far>3</far>
+        </clip>
+        <noise>
+          <type>gaussian</type>
+          <mean>0.0</mean>
+          <stddev>0.007</stddev>
+        </noise>
+      </camera>
+      <!-- Plugin to publish images and camera info to ROS topics -->
+      <plugin name="${camera_pos}_camera_controller" filename="libgazebo_ros_camera.so">
+        <alwaysOn>true</alwaysOn>
+        <updateRate>0.0</updateRate>
+        <cameraName>${camera_pos}_camera</cameraName>
+        <imageTopicName>image_raw</imageTopicName>
+        <cameraInfoTopicName>camera_info</cameraInfoTopicName>
+        <frameName>/${camera_pos}_rs_gazebo_camera_frame</frameName>
+        <hackBaseline>0.07</hackBaseline>
+        <distortionK1>0.0</distortionK1>
+        <distortionK2>0.0</distortionK2>
+        <distortionK3>0.0</distortionK3>
+        <distortionT1>0.0</distortionT1>
+        <distortionT2>0.0</distortionT2>
+      </plugin>
+    </sensor>
+  </gazebo>
     <link name="${camera_pos}_rs_depth_optical_frame">
     </link>

Commit message: setup drone to be namespaced

File: linorobot2_description/urdf/mecanum_properties.urdf.xacro (robot description, xacro)
@@ -4,5 +4,5 @@
   <xacro:property name="base_width" value="0.495" />
   <xacro:property name="base_height" value="0.116" />
-  <xacro:property name="base_mass" value="30" />
+  <!-- <xacro:property name="base_mass" value="30" />
   <xacro:property name="wheel_radius" value="0.07162" />
   <xacro:property name="wheel_width" value="0.05" />
@@ -17,4 +17,4 @@
   <xacro:property name="depth_sensor_pose">
     <origin xyz="0.2375 0 0.06" rpy="0 0 0"/>
-  </xacro:property>
+  </xacro:property> -->
 </robot>

File: linorobot2_description/urdf/robots/camera.urdf.xacro (robot description, xacro)
@@ -1,5 +1,5 @@
 <?xml version="1.0"?>
 <robot name="linorobot2_mecanum" xmlns:xacro="http://ros.org/wiki/xacro">
-  <xacro:macro name="camera" params="camera_pos x y z r_rs p_rs yaw_rs r_cam p_cam yaw_cam">
+  <xacro:macro name="camera" params="namespace camera_pos x y z r_rs p_rs yaw_rs r_cam p_cam yaw_cam">
     <gazebo reference="${camera_pos}_gazebo_camera_frame">
     <sensor type="depth" name="${camera_pos}_camera">
@@ -22,6 +22,9 @@
         </noise>
       </camera>
-      <!-- Plugin to publish images and camera info to ROS topics -->
       <plugin name="${camera_pos}_camera_controller" filename="libgazebo_ros_camera.so">
+        <ros>
+            <namespace>${namespace}</namespace>
+            <!-- TODO - remap gazebo topics to ros topics that match the topics on a physical realsense -->
+        </ros>
         <alwaysOn>true</alwaysOn>
         <updateRate>0.0</updateRate>
@@ -41,5 +44,4 @@
     <link name="${camera_pos}_rs_depth_optical_frame">
     </link>
-    <!-- This is the position that a realsense camera would be mounted on the robot -->
     <joint
       name="base_link_to_${camera_pos}_rs" type="fixed">

File: linorobot2_description/urdf/robots/mecanum_libplanar.urdf.xacro (robot description, xacro)
@@ -1,4 +1,5 @@
 <?xml version="1.0"?>
-<robot name="linorobot2" xmlns:xacro="http://ros.org/wiki/xacro">
+<robot name="linorobot2" xmlns:xacro="http://www.ros.org/wiki/xacro">
+  <xacro:arg name="namespace" default="drone0"/>
   <xacro:include filename="$(find linorobot2_description)/urdf/mecanum_properties.urdf.xacro" />
   <xacro:include filename="$(find linorobot2_description)/urdf/mech/base.urdf.xacro" />
@@ -8,23 +9,27 @@
   <xacro:include filename="$(find linorobot2_description)/urdf/robots/camera.urdf.xacro" />
   <xacro:property name="rs_height" value="${base_height/2 + 0.05}" />
-  <xacro:camera camera_pos="front" x="0.410335" y="0" z="${rs_height}"
-                                   r_rs= "-1.57" p_rs="0" yaw_rs="-1.57"
-                                   r_cam="0" p_cam="0" yaw_cam="0"
-                                   />
-  <xacro:camera camera_pos="left" x="0.0" y="0.247" z="${rs_height}"
-                                  r_rs="-1.57" p_rs="0.0" yaw_rs="0"
-                                  r_cam="0" p_cam="0" yaw_cam="1.57"
-                                  />
-  <xacro:camera camera_pos="rear" x="-0.41" y="0.0" z="${rs_height}"
-                                  r_rs="-1.57" p_rs="0" yaw_rs="1.57"
-                                  r_cam="0" p_cam="0" yaw_cam="3.14"
-                                  />
-  <xacro:camera camera_pos="right" x="0" y="-0.247" z="${rs_height}"
-                                  r_rs="-1.57" p_rs="0" yaw_rs="3.14"
-                                  r_cam="0" p_cam="0" yaw_cam="-1.57"
-                                  />
+  <xacro:camera namespace="$(arg namespace)" camera_pos="front"
+                x="0.410335" y="0" z="${rs_height}"
+                r_rs= "-1.57" p_rs="0" yaw_rs="-1.57"
+                r_cam="0" p_cam="0" yaw_cam="0"/>
+  <xacro:camera namespace="$(arg namespace)" camera_pos="left"
+                x="0.0" y="0.247" z="${rs_height}"
+                r_rs="-1.57" p_rs="0.0" yaw_rs="0"
+                r_cam="0" p_cam="0" yaw_cam="1.57"
+  />
+  <xacro:camera namespace="$(arg namespace)" camera_pos="rear"
+                x="-0.41" y="0.0" z="${rs_height}"
+                r_rs="-1.57" p_rs="0" yaw_rs="1.57"
+                r_cam="0" p_cam="0" yaw_cam="3.14"
+  />
+  <xacro:camera namespace="$(arg namespace)" camera_pos="right"
+                x="0" y="-0.247" z="${rs_height}"
+                r_rs="-1.57" p_rs="0" yaw_rs="3.14"
+                r_cam="0" p_cam="0" yaw_cam="-1.57"
+  />
   <gazebo>
     <plugin name="mecanum_wheel_mimic" filename="libgazebo_ros_planar_move.so">
       <ros>
+        <namespace>$(arg namespace)</namespace>
         <remapping>odom:=/odom_unscaled</remapping>
         <remapping>cmd_vel:=/cmd_vel_scaled</remapping>
