Commit message: All 4 realsenses have their points transformed to the base link properly now

File: linorobot2_description/urdf/robots/camera.urdf.xacro (robot description, xacro)
@@ -1,5 +1,5 @@
 <?xml version="1.0"?>
 <robot name="linorobot2_mecanum" xmlns:xacro="http://ros.org/wiki/xacro">
-  <xacro:macro name="camera" params="camera_pos x y z r_rs p_rs yaw_rs">
+  <xacro:macro name="camera" params="camera_pos x y z r_rs p_rs yaw_rs r_cam p_cam yaw_cam">
     <gazebo reference="${camera_pos}_gazebo_camera_frame">
       <sensor type="depth" name="${camera_pos}_camera">
@@ -54,6 +54,6 @@
       name="base_link_to_${camera_pos}_gazebo_camera_frame" type="fixed">
       <origin
-        xyz="0.3 0 0"
-        rpy="0 0 0" />
+        xyz="${x} ${y} ${z}"
+        rpy="${r_cam} ${p_cam} ${yaw_cam}" />
       <parent link="base_link" />
       <child link="${camera_pos}_gazebo_camera_frame" />

File: linorobot2_description/urdf/robots/mecanum_libplanar.urdf.xacro (robot description, xacro)
@@ -11,12 +11,20 @@
   <link name="base_link">
   </link>
-  <xacro:camera camera_pos="front" x="0.410335" y="0" z="0.3"
-                                   r_rs= "-1.57" p_rs="0" yaw_rs="-1.57" />
-  <!-- <xacro:camera camera_pos="left" x="0.0" y="0.247" z="0.089"
-                                  r_rs="-1.57" p_rs="0.0" yaw_rs="0"/>
+  <xacro:camera camera_pos="front" x="0.410335" y="0" z="0.089"
+                                   r_rs= "-1.57" p_rs="0" yaw_rs="-1.57"
+                                   r_cam="0" p_cam="0" yaw_cam="0"
+                                   />
+  <xacro:camera camera_pos="left" x="0.0" y="0.247" z="0.089"
+                                  r_rs="-1.57" p_rs="0.0" yaw_rs="0"
+                                  r_cam="0" p_cam="0" yaw_cam="1.57"
+                                  />
   <xacro:camera camera_pos="rear" x="-0.41" y="0.0" z="0.089"
-                                  r_rs="-1.57" p_rs="0" yaw_rs="1.57" />
+                                  r_rs="-1.57" p_rs="0" yaw_rs="1.57"
+                                  r_cam="0" p_cam="0" yaw_cam="3.14"
+                                  />
   <xacro:camera camera_pos="right" x="0" y="-0.247" z="0.089"
-                                  r_rs="-1.57" p_rs="0" yaw_rs="3.14"/> -->
+                                  r_rs="-1.57" p_rs="0" yaw_rs="3.14"
+                                  r_cam="0" p_cam="0" yaw_cam="-1.57"
+                                  />
   <!-- <gazebo>
     <plugin name="mecanum_wheel_mimic" filename="libgazebo_ros_planar_move.so">

Commit message: Updated camera names to match physical realsenses

File: linorobot2_description/urdf/robots/camera.urdf.xacro (robot description, xacro)
@@ -2,4 +2,5 @@
 <robot name="linorobot2_mecanum" xmlns:xacro="http://ros.org/wiki/xacro">
   <xacro:macro name="camera" params="namespace camera_pos x y z r_rs p_rs yaw_rs r_cam p_cam yaw_cam">
+    <xacro:property name="rs_pcl_topic" value="/${namespace}/${camera_pos}_rs/${camera_pos}_rs/depth/color/points" />
     <gazebo reference="${namespace}_${camera_pos}_gazebo_camera_frame">
     <sensor type="depth" name="${camera_pos}_rs">
@@ -25,13 +26,13 @@
         <ros>
             <namespace>${namespace}</namespace>
-            <remap>points:=${camera_pos}_rs/depth/color/points</remap>
-            <!-- TODO - remap gazebo topics to ros topics that match the topics on a physical realsense -->
+            <remapping>/${namespace}/${camera_pos}_rs/points:=${rs_pcl_topic}</remapping>
         </ros>
         <alwaysOn>true</alwaysOn>
         <updateRate>0.0</updateRate>
-        <cameraName>${camera_pos}_camera</cameraName>
+        <cameraName>${namespace}_${camera_pos}_camera</cameraName>
+        <pointsTopicName>points</pointsTopicName>
         <imageTopicName>image_raw</imageTopicName>
         <cameraInfoTopicName>camera_info</cameraInfoTopicName>
-        <frameName>${namespace}_${camera_pos}_rs_gazebo_camera_frame</frameName>
+        <frameName>/${namespace}_${camera_pos}_rs_gazebo_camera_frame</frameName>
         <hackBaseline>0.07</hackBaseline>
         <distortionK1>0.0</distortionK1>
