Commit message: description package cleanup

File: antdrone_description/urdf/base.urdf.xacro (robot description, xacro)
@@ -2,5 +2,5 @@
 <robot xmlns:xacro="http://ros.org/wiki/xacro">
   <xacro:macro name="base" params="namespace length width height">
-    <!-- Beware changing masses or inertias of the base link. It will affect the robot's motion. -->
+    <!-- Beware of changing masses or inertias of the base link. It will affect the robot's motion. -->
     <!-- Gazebos planar move model moves the robot at a different velocity than requested, but publishes the requested velocity in odometry. -->
     <!-- A linear transformation between desired and actual velocity is applied to the velocity going into Gazebo planar movement, and to the odom coming out of Gazebo planar movement -->

File: antdrone_description/urdf/camera.urdf.xacro (robot description, xacro)
@@ -15,5 +15,7 @@
         <clip>
           <near>0.05</near>
-          <far>5</far> <!--  Be sure to set this greater than the max value of the cropbox distance cutoff, the camera generates a grey plane at this distance that will be interpreted as an obstacle-->
+          <!--  Be sure to set far clip greater than cropbox node's cutoff distance.
+            The camera generates a grey plane at this distance that will be interpreted in nav2 as an obstacle-->
+          <far>5</far>
         </clip>
         <noise>

File: antdrone_description/urdf/mecanum_libplanar.urdf.xacro (robot description, xacro)
@@ -3,9 +3,6 @@
   <xacro:arg name="namespace" default=""/>
   <xacro:include filename="$(find antdrone_description)/urdf/mecanum_properties.urdf.xacro" />
-  <xacro:include filename="$(find antdrone_description)/urdf/mech/base.urdf.xacro" />
-  <xacro:include filename="$(find antdrone_description)/urdf/mech/mecanum_wheel_left_fixed.urdf.xacro" />
-  <xacro:include filename="$(find antdrone_description)/urdf/mech/end_channel.urdf.xacro" />
-  <xacro:include filename="$(find antdrone_description)/urdf/mech/side_channel.urdf.xacro" />
-  <xacro:include filename="$(find antdrone_description)/urdf/robots/camera.urdf.xacro" />
+  <xacro:include filename="$(find antdrone_description)/urdf/base.urdf.xacro" />
+  <xacro:include filename="$(find antdrone_description)/urdf/camera.urdf.xacro" />
   <xacro:property name="rs_height" value="${base_height/2 + 0.05}" />
   <xacro:camera namespace="$(arg namespace)" camera_pos="front"

File: antdrone_description/urdf/mecanum_properties.urdf.xacro (robot description, xacro)
@@ -4,17 +4,3 @@
   <xacro:property name="base_width" value="0.495" />
   <xacro:property name="base_height" value="0.116" />
-  <!-- <xacro:property name="base_mass" value="30" />
-  <xacro:property name="wheel_radius" value="0.07162" />
-  <xacro:property name="wheel_width" value="0.05" />
-  <xacro:property name="wheel_pos_x" value="0.25857" />
-  <xacro:property name="wheel_pos_y" value="0.19355" />
-  <xacro:property name="wheel_pos_z" value="0.0019" />
-  <xacro:property name="wheel_mass" value="2.0" />
-  <xacro:property name="wheel_torque" value="20" />
-  <xacro:property name="laser_pose">
-    <origin xyz="-0.0475 0 0.125" rpy="0 0 0"/>
-  </xacro:property>
-  <xacro:property name="depth_sensor_pose">
-    <origin xyz="0.2375 0 0.06" rpy="0 0 0"/>
-  </xacro:property> -->
 </robot>

Commit message: Resolved need for velocity scaling with velocities sent to gazebo lib planar movement plugin. Simply reduced friction of drone base link

File: antdrone_description/urdf/base.urdf.xacro (robot description, xacro)
@@ -21,12 +21,12 @@
       <inertial>
         <origin xyz="0 0 0" rpy="0 0 0"/>
-        <mass value="20"/> <!-- Small, non-zero mass -->
+        <mass value="10"/> <!-- Small, non-zero mass -->
         <inertia
-          ixx="1.14"
+          ixx="0.57"
           ixy="-4.74983711945811E-18"
           ixz="-1.80635263223563E-18"
-          iyy="1.53"
+          iyy="0.765"
           iyz="6.42624983676543E-18"
-          izz="0.43" />
+          izz="0.215" />
       </inertial>
     </link>
@@ -35,6 +35,6 @@
     <turnGravityOff>false</turnGravityOff>
     <selfCollide>true</selfCollide>
-    <mu1>0.2</mu1>
-    <mu2>0.2</mu2>
+    <mu1>0.05</mu1>
+    <mu2>0.05</mu2>
   </gazebo>
   <link name="${namespace}_attachment_point">

Commit message: Added gz spawn in seperate container, in this repo instead of fleet demos repo, so that it can be re-used in drone-only simulations

File: antdrone_description/urdf/base.urdf.xacro (robot description, xacro)
@@ -1,6 +1,7 @@
 <?xml version="1.0"?>
 <robot xmlns:xacro="http://ros.org/wiki/xacro">
-  <xacro:macro name="base" params="namespace length width height">
-    <link name="${namespace}_base_link">
+  <xacro:macro name="base" params="drone_name length width height">
+    <!-- Links must have drone_name at the start in case there is another drone -->
+    <link name="${drone_name}_base_link">
       <visual>
         <origin xyz="0 0 0" rpy="0 0 0"/>
@@ -27,5 +28,5 @@
       </inertial>
     </link>
-  <gazebo reference="${namespace}_base_link">
+  <gazebo reference="${drone_name}_base_link">
     <material>Gazebo/White</material>
     <turnGravityOff>false</turnGravityOff>
@@ -35,5 +36,5 @@
     <mu2>0.05</mu2>
   </gazebo>
-  <link name="${namespace}_attachment_point">
+  <link name="${drone_name}_attachment_point">
       <inertial>
         <origin xyz="0 0 0" rpy="0 0 0"/>
@@ -48,15 +49,15 @@
       </inertial>
     </link>
-  <gazebo reference="${namespace}_attachment_point">
+  <!-- <gazebo reference="${drone_name}_attachment_point">
     <material>Gazebo/Gray</material>
     <turnGravityOff>false</turnGravityOff>
     <selfCollide>true</selfCollide>
-  </gazebo>
-  <joint name="${namespace}_attachment_to_base" type="fixed">
-    <parent link="${namespace}_base_link"/>
-    <child link="${namespace}_attachment_point"/>
+  </gazebo> -->
+  <joint name="${drone_name}_attachment_to_base" type="fixed">
+    <parent link="${drone_name}_base_link"/>
+    <child link="${drone_name}_attachment_point"/>
     <origin xyz="0 0 0.6" rpy="0 0 1.57"/>
   </joint>
-  <gazebo reference='${namespace}_attachment_to_base'>
+  <gazebo reference='${drone_name}_attachment_to_base'>
     <preserveFixedJoint>true</preserveFixedJoint>
   </gazebo>

File: antdrone_description/urdf/camera.urdf.xacro (robot description, xacro)
@@ -1,68 +1,67 @@
 <?xml version="1.0"?>
 <robot name="antdrone_camera" xmlns:xacro="http://ros.org/wiki/xacro">
-  <xacro:macro name="camera" params="namespace camera_pos x y z r_rs p_rs yaw_rs r_cam p_cam yaw_cam">
-    <xacro:property name="rs_pcl_topic" value="/${namespace}/${camera_pos}_rs/${camera_pos}_rs/depth/color/points" />
-    <gazebo reference="${namespace}_${camera_pos}_gazebo_camera_frame">
-    <sensor type="depth" name="${camera_pos}_rs">
-      <update_rate>15.0</update_rate> <!-- Gazebo does not necessarily respect this update rate when publishing the camera data to ros2 -->
-      <camera>
-        <horizontal_fov>1.517</horizontal_fov>
-        <image>
-          <width>100</width>
-          <height>56</height>
-          <format>R8G8B8</format>
-        </image>
-        <clip>
-          <near>0.05</near>
-          <!--  Be sure to set far clip greater than cropbox node's cutoff distance.
-            The camera generates a grey plane at this distance that will be interpreted in nav2 as an obstacle-->
-          <far>5</far>
-        </clip>
-        <noise>
-          <type>gaussian</type>
-          <mean>0.0</mean>
-          <stddev>0.007</stddev>
-        </noise>
-      </camera>
-      <plugin name="${camera_pos}_camera_controller" filename="libgazebo_ros_camera.so">
-        <ros>
-            <namespace>${namespace}</namespace>
-            <remapping>/${namespace}/${camera_pos}_rs/points:=${rs_pcl_topic}</remapping>
-        </ros>
-        <alwaysOn>true</alwaysOn>
-        <updateRate>0.0</updateRate>
-        <cameraName>${namespace}_${camera_pos}_camera</cameraName>
-        <pointsTopicName>points</pointsTopicName>
-        <imageTopicName>image_raw</imageTopicName>
-        <cameraInfoTopicName>camera_info</cameraInfoTopicName>
-        <frameName>/${namespace}_${camera_pos}_rs_gazebo_camera_frame</frameName>
-        <hackBaseline>0.07</hackBaseline>
-        <distortionK1>0.0</distortionK1>
-        <distortionK2>0.0</distortionK2>
-        <distortionK3>0.0</distortionK3>
-        <distortionT1>0.0</distortionT1>
-        <distortionT2>0.0</distortionT2>
-      </plugin>
-    </sensor>
-  </gazebo>
-    <link name="${namespace}_${camera_pos}_rs_depth_optical_frame">
+  <xacro:macro name="camera" params="drone_name camera_pos x y z r_rs p_rs yaw_rs r_cam p_cam yaw_cam">
+    <gazebo reference="${drone_name}_${camera_pos}_gazebo_camera_frame">
+      <sensor type="depth" name="${camera_pos}_rs">
+        <update_rate>15.0</update_rate> <!-- Gazebo does not necessarily respect this update rate when publishing the camera data to ros2 -->
+        <camera>
+          <horizontal_fov>1.517</horizontal_fov>
+          <image>
+            <width>100</width>
+            <height>56</height>
+            <format>R8G8B8</format>
+          </image>
+          <clip>
+            <near>0.05</near>
+            <!--  Be sure to set far clip greater than cropbox node's cutoff distance.
+              The camera generates a grey plane at this distance that will be interpreted in nav2 as an obstacle-->
+            <far>5</far>
+          </clip>
+          <noise>
+            <type>gaussian</type>
+            <mean>0.0</mean>
+            <stddev>0.007</stddev>
+          </noise>
+        </camera>
+        <plugin name="${camera_pos}_camera_controller" filename="libgazebo_ros_camera.so">
+          <ros>
+              <namespace>${drone_name}</namespace>
+          </ros>
+          <alwaysOn>true</alwaysOn>
+          <updateRate>0.0</updateRate>
+          <cameraName>${camera_pos}_camera</cameraName>
+          <pointsTopicName>points</pointsTopicName>
+          <imageTopicName>image_raw</imageTopicName>
+          <cameraInfoTopicName>camera_info</cameraInfoTopicName>
+          <frameName>${camera_pos}_rs_gazebo_camera_frame</frameName>
+          <hackBaseline>0.07</hackBaseline>
+          <distortionK1>0.0</distortionK1>
+          <distortionK2>0.0</distortionK2>
+          <distortionK3>0.0</distortionK3>
+          <distortionT1>0.0</distortionT1>
+          <distortionT2>0.0</distortionT2>
+        </plugin>
+      </sensor>
+    </gazebo>
+    <!-- Links must have drone_name at the start in case there is another drone -->
+    <link name="${drone_name}_${camera_pos}_rs_depth_optical_frame">
     </link>
     <joint
-      name="${namespace}_base_link_to_${camera_pos}_rs" type="fixed">
+      name="${drone_name}_base_link_to_${camera_pos}_rs" type="fixed">
       <origin
         xyz="${x} ${y} ${z}"
         rpy="${r_rs} ${p_rs} ${yaw_rs}" />
-      <parent link="${namespace}_base_link" />
-      <child link="${namespace}_${camera_pos}_rs_depth_optical_frame" />
+      <parent link="${drone_name}_base_link" />
+      <child link="${drone_name}_${camera_pos}_rs_depth_optical_frame" />
     </joint>
-    <link name="${namespace}_${camera_pos}_gazebo_camera_frame">
+    <link name="${drone_name}_${camera_pos}_gazebo_camera_frame">
     </link>
     <joint
-      name="${namespace}_base_link_to_${camera_pos}_gazebo_camera_frame" type="fixed">
+      name="${drone_name}_base_link_to_${camera_pos}_gazebo_camera_frame" type="fixed">
       <origin
         xyz="${x} ${y} ${z}"
         rpy="${r_cam} ${p_cam} ${yaw_cam}" />
-      <parent link="${namespace}_base_link" />
-      <child link="${namespace}_${camera_pos}_gazebo_camera_frame" />
+      <parent link="${drone_name}_base_link" />
+      <child link="${drone_name}_${camera_pos}_gazebo_camera_frame" />
     </joint>
   </xacro:macro>

File: antdrone_description/urdf/mecanum_libplanar.urdf.xacro (robot description, xacro)
@@ -6,19 +6,19 @@
   <xacro:include filename="$(find antdrone_description)/urdf/camera.urdf.xacro" />
   <xacro:property name="rs_height" value="${base_height/2 + 0.05}" />
-  <xacro:camera namespace="$(arg namespace)" camera_pos="front"
+  <xacro:camera drone_name="$(arg namespace)" camera_pos="front"
                 x="0.410335" y="0" z="${rs_height}"
                 r_rs= "-1.57" p_rs="0" yaw_rs="-1.57"
                 r_cam="0" p_cam="0" yaw_cam="0"/>
-  <xacro:camera namespace="$(arg namespace)" camera_pos="left"
+  <xacro:camera drone_name="$(arg namespace)" camera_pos="left"
                 x="0.0" y="0.247" z="${rs_height}"
                 r_rs="-1.57" p_rs="0.0" yaw_rs="0"
                 r_cam="0" p_cam="0" yaw_cam="1.57"
   />
-  <xacro:camera namespace="$(arg namespace)" camera_pos="rear"
+  <xacro:camera drone_name="$(arg namespace)" camera_pos="rear"
                 x="-0.41" y="0.0" z="${rs_height}"
                 r_rs="-1.57" p_rs="0" yaw_rs="1.57"
                 r_cam="0" p_cam="0" yaw_cam="3.14"
   />
-  <xacro:camera namespace="$(arg namespace)" camera_pos="right"
+  <xacro:camera drone_name="$(arg namespace)" camera_pos="right"
                 x="0" y="-0.247" z="${rs_height}"
                 r_rs="-1.57" p_rs="0" yaw_rs="3.14"
@@ -44,5 +44,5 @@
   </gazebo>
   <xacro:base
-    namespace="$(arg namespace)"
+    drone_name="$(arg namespace)"
     length="${base_length}"
     width="${base_width}"

Commit message: Simplified frame naming and changed AMCL to have initial pose from config rather than service call

File: antdrone_description/urdf/base.urdf.xacro (robot description, xacro)
@@ -2,6 +2,5 @@
 <robot xmlns:xacro="http://ros.org/wiki/xacro">
   <xacro:macro name="base" params="drone_name length width height">
-    <!-- Links must have drone_name at the start in case there is another drone -->
-    <link name="${drone_name}_base_link">
+    <link name="base_link">
       <visual>
         <origin xyz="0 0 0" rpy="0 0 0"/>
@@ -28,5 +27,5 @@
       </inertial>
     </link>
-  <gazebo reference="${drone_name}_base_link">
+  <gazebo reference="base_link">
     <material>Gazebo/White</material>
     <turnGravityOff>false</turnGravityOff>
@@ -36,5 +35,5 @@
     <mu2>0.05</mu2>
   </gazebo>
-  <link name="${drone_name}_attachment_point">
+  <link name="attachment_point">
       <inertial>
         <origin xyz="0 0 0" rpy="0 0 0"/>
@@ -49,15 +48,10 @@
       </inertial>
     </link>
-  <!-- <gazebo reference="${drone_name}_attachment_point">
-    <material>Gazebo/Gray</material>
-    <turnGravityOff>false</turnGravityOff>
-    <selfCollide>true</selfCollide>
-  </gazebo> -->
-  <joint name="${drone_name}_attachment_to_base" type="fixed">
-    <parent link="${drone_name}_base_link"/>
-    <child link="${drone_name}_attachment_point"/>
+  <joint name="attachment_to_base" type="fixed">
+    <parent link="base_link"/>
+    <child link="attachment_point"/>
     <origin xyz="0 0 0.6" rpy="0 0 1.57"/>
   </joint>
-  <gazebo reference='${drone_name}_attachment_to_base'>
+  <gazebo reference='attachment_to_base'>
     <preserveFixedJoint>true</preserveFixedJoint>
   </gazebo>

File: antdrone_description/urdf/camera.urdf.xacro (robot description, xacro)
@@ -2,5 +2,5 @@
 <robot name="antdrone_camera" xmlns:xacro="http://ros.org/wiki/xacro">
   <xacro:macro name="camera" params="drone_name camera_pos x y z r_rs p_rs yaw_rs r_cam p_cam yaw_cam">
-    <gazebo reference="${drone_name}_${camera_pos}_gazebo_camera_frame">
+    <gazebo reference="${camera_pos}_gazebo_camera_frame">
       <sensor type="depth" name="${camera_pos}_rs">
         <update_rate>15.0</update_rate> <!-- Gazebo does not necessarily respect this update rate when publishing the camera data to ros2 -->
@@ -44,24 +44,23 @@
       </sensor>
     </gazebo>
-    <!-- Links must have drone_name at the start in case there is another drone -->
-    <link name="${drone_name}_${camera_pos}_rs_depth_optical_frame">
+    <link name="${camera_pos}_rs_depth_optical_frame">
     </link>
     <joint
-      name="${drone_name}_base_link_to_${camera_pos}_rs" type="fixed">
+      name="base_link_to_${camera_pos}_rs" type="fixed">
       <origin
         xyz="${x} ${y} ${z}"
         rpy="${r_rs} ${p_rs} ${yaw_rs}" />
-      <parent link="${drone_name}_base_link" />
-      <child link="${drone_name}_${camera_pos}_rs_depth_optical_frame" />
+      <parent link="base_link" />
+      <child link="${camera_pos}_rs_depth_optical_frame" />
     </joint>
-    <link name="${drone_name}_${camera_pos}_gazebo_camera_frame">
+    <link name="${camera_pos}_gazebo_camera_frame">
     </link>
     <joint
-      name="${drone_name}_base_link_to_${camera_pos}_gazebo_camera_frame" type="fixed">
+      name="base_link_to_${camera_pos}_gazebo_camera_frame" type="fixed">
       <origin
         xyz="${x} ${y} ${z}"
         rpy="${r_cam} ${p_cam} ${yaw_cam}" />
-      <parent link="${drone_name}_base_link" />
-      <child link="${drone_name}_${camera_pos}_gazebo_camera_frame" />
+      <parent link="base_link" />
+      <child link="${camera_pos}_gazebo_camera_frame" />
     </joint>
   </xacro:macro>

File: antdrone_description/urdf/mecanum_libplanar.urdf.xacro (robot description, xacro)
@@ -1,24 +1,24 @@
 <?xml version="1.0"?>
 <robot name="antdrone" xmlns:xacro="http://www.ros.org/wiki/xacro">
-  <xacro:arg name="namespace" default=""/>
+  <xacro:arg name="drone_name" default=""/>
   <xacro:include filename="$(find antdrone_description)/urdf/mecanum_properties.urdf.xacro" />
   <xacro:include filename="$(find antdrone_description)/urdf/base.urdf.xacro" />
   <xacro:include filename="$(find antdrone_description)/urdf/camera.urdf.xacro" />
   <xacro:property name="rs_height" value="${base_height/2 + 0.05}" />
-  <xacro:camera drone_name="$(arg namespace)" camera_pos="front"
+  <xacro:camera drone_name="$(arg drone_name)" camera_pos="front"
                 x="0.410335" y="0" z="${rs_height}"
                 r_rs= "-1.57" p_rs="0" yaw_rs="-1.57"
                 r_cam="0" p_cam="0" yaw_cam="0"/>
-  <xacro:camera drone_name="$(arg namespace)" camera_pos="left"
+  <xacro:camera drone_name="$(arg drone_name)" camera_pos="left"
                 x="0.0" y="0.247" z="${rs_height}"
                 r_rs="-1.57" p_rs="0.0" yaw_rs="0"
                 r_cam="0" p_cam="0" yaw_cam="1.57"
   />
-  <xacro:camera drone_name="$(arg namespace)" camera_pos="rear"
+  <xacro:camera drone_name="$(arg drone_name)" camera_pos="rear"
                 x="-0.41" y="0.0" z="${rs_height}"
                 r_rs="-1.57" p_rs="0" yaw_rs="1.57"
                 r_cam="0" p_cam="0" yaw_cam="3.14"
   />
-  <xacro:camera drone_name="$(arg namespace)" camera_pos="right"
+  <xacro:camera drone_name="$(arg drone_name)" camera_pos="right"
                 x="0" y="-0.247" z="${rs_height}"
                 r_rs="-1.57" p_rs="0" yaw_rs="3.14"
@@ -28,13 +28,15 @@
     <plugin name="mecanum_wheel_mimic" filename="libgazebo_ros_planar_move.so">
       <ros>
-        <!-- Since all robots exist in gazebo in the MAIN_ROS_DOMAIN_ID, their topics must be namespaced. -->
-        <!-- Namespaces are removed when topics are domain-bridged to each robot, to mimic topic names on physical robots -->
-        <namespace>$(arg namespace)</namespace>
+        <!-- The planar move plugin publishes each robot's odom -> base link transform in the ROS DOMAIN ID of gazebo,
+          so each robot's odometry frame must be prepended by the robot's name. The prepended robot name is stripped out
+          when the tf is bridged into the robots ROS domain ID.
+         -->
+        <namespace>$(arg drone_name)</namespace>
       </ros>
       <command_topic>cmd_vel</command_topic>
       <odometry_topic>odom</odometry_topic>
-      <odometry_frame>$(arg namespace)_odom</odometry_frame>
+      <odometry_frame>$(arg drone_name)_odom</odometry_frame>
       <odometry_rate>15.0</odometry_rate>
-      <robot_base_frame>$(arg namespace)_base_link</robot_base_frame>
+      <robot_base_frame>$(arg drone_name)_base_link</robot_base_frame>
       <publish_odom>true</publish_odom>
       <publish_odom_tf>true</publish_odom_tf>
@@ -44,5 +46,5 @@
   </gazebo>
   <xacro:base
-    drone_name="$(arg namespace)"
+    drone_name="$(arg drone_name)"
     length="${base_length}"
     width="${base_width}"

Commit message: Got drone sensing april tags on worker, now to figure out optimal placement of tags on worker and extra camera on drone

File: antdrone_description/urdf/base.urdf.xacro (robot description, xacro)
@@ -28,5 +28,5 @@
     </link>
   <gazebo reference="base_link">
-    <material>Gazebo/White</material>
+    <material>Gazebo/Orange</material>
     <turnGravityOff>false</turnGravityOff>
     <selfCollide>true</selfCollide>

File: antdrone_description/urdf/camera.urdf.xacro (robot description, xacro)
@@ -8,10 +8,12 @@
           <horizontal_fov>1.517</horizontal_fov>
           <image>
-            <width>100</width>
-            <height>56</height>
+            <!-- Set width & height to match settings on physical realsense -->
+            <width>640</width>
+            <height>480</height>
             <format>R8G8B8</format>
           </image>
           <clip>
-            <near>0.05</near>
+            <!-- Physical realsense cuts off around 10cm, sim camera seems to cutoff at 30cm no matter what. -->
+            <near>0.1</near>
             <!--  Be sure to set far clip greater than cropbox node's cutoff distance.
               The camera generates a grey plane at this distance that will be interpreted in nav2 as an obstacle-->
