Commit message: realsense cameras positioned correctly in sim to match camera heights of physical realsenses

File: antdrone_description/urdf/base.urdf.xacro (robot description, xacro)
@@ -4,5 +4,5 @@
     <link name="base_link">
       <visual>
-        <origin xyz="0 0 0" rpy="0 0 0"/>
+        <origin xyz="0 0 ${height/2}" rpy="0 0 0"/>
         <geometry>
           <box size="${length} ${width} ${height}"/>
@@ -10,5 +10,5 @@
       </visual>
       <collision>
-        <origin xyz="0 0 0" rpy="0 0 0"/>
+        <origin xyz="0 0 ${height/2}" rpy="0 0 0"/>
         <geometry>
           <box size="${length} ${width} ${height}"/>
@@ -16,5 +16,5 @@
       </collision>
       <inertial>
-        <origin xyz="0 0 0" rpy="0 0 0"/>
+        <origin xyz="0 0 ${height/2}" rpy="0 0 0"/>
         <mass value="10"/> <!-- Small, non-zero mass -->
         <inertia

File: antdrone_description/urdf/mecanum_libplanar.urdf.xacro (robot description, xacro)
@@ -5,20 +5,25 @@
   <xacro:include filename="$(find antdrone_description)/urdf/base.urdf.xacro" />
   <xacro:include filename="$(find antdrone_description)/urdf/camera.urdf.xacro" />
-  <xacro:property name="rs_height" value="${0.37 - base_height/2}" />
-  <xacro:camera drone_name="$(arg drone_name)" camera_pos="front"
-                x="${base_length/2 - 0.0575}" y="-0.195" z="${rs_height}"
+  <xacro:include filename="$(find antdrone_description)/urdf/rs.urdf.xacro" />
+  <xacro:property name="rs_height" value="${base_height + 0.04}" />
+  <xacro:camera drone_name="$(arg drone_name)" camera_name="apriltag_cam"
+                x="${base_length/2 - 0.0575}" y="-0.195" z="0.37"
                 r_rs= "-1.57" p_rs="0" yaw_rs="${(60-90)/180*3.14}"
                 r_cam="0" p_cam="0" yaw_cam="${60/180*3.14}"/>
-  <xacro:camera drone_name="$(arg drone_name)" camera_pos="left"
+  <xacro:rs drone_name="$(arg drone_name)" camera_name="front_rs"
+                x="0.41" y="0.0" z="${rs_height}"
+                r_rs= "-1.57" p_rs="0" yaw_rs="-1.57"
+                r_cam="0" p_cam="0" yaw_cam="0"/>
+  <xacro:rs drone_name="$(arg drone_name)" camera_name="left_rs"
                 x="0.0" y="0.247" z="${rs_height}"
                 r_rs="-1.57" p_rs="0.0" yaw_rs="0"
                 r_cam="0" p_cam="0" yaw_cam="1.57"
   />
-  <xacro:camera drone_name="$(arg drone_name)" camera_pos="rear"
+  <xacro:rs drone_name="$(arg drone_name)" camera_name="rear_rs"
                 x="-0.41" y="0.0" z="${rs_height}"
                 r_rs="-1.57" p_rs="0" yaw_rs="1.57"
                 r_cam="0" p_cam="0" yaw_cam="3.14"
   />
-  <xacro:camera drone_name="$(arg drone_name)" camera_pos="right"
+  <xacro:rs drone_name="$(arg drone_name)" camera_name="right_rs"
                 x="0" y="-0.247" z="${rs_height}"
                 r_rs="-1.57" p_rs="0" yaw_rs="3.14"

File: antdrone_description/urdf/mecanum_properties.urdf.xacro (robot description, xacro)
@@ -3,4 +3,4 @@
   <xacro:property name="base_length" value="0.82" />
   <xacro:property name="base_width" value="0.495" />
-  <xacro:property name="base_height" value="0.116" />
+  <xacro:property name="base_height" value="0.116" /> <!-- 0.116 is height from ground to top of drone rail-->
 </robot>

File: antdrone_description/urdf/rs.urdf.xacro (robot description, xacro)
@@ -1,17 +1,18 @@
 <?xml version="1.0"?>
 <robot name="antdrone_camera" xmlns:xacro="http://ros.org/wiki/xacro">
-  <xacro:macro name="camera" params="drone_name camera_name x y z r_rs p_rs yaw_rs r_cam p_cam yaw_cam">
+  <xacro:macro name="rs" params="drone_name camera_name x y z r_rs p_rs yaw_rs r_cam p_cam yaw_cam">
     <gazebo reference="${camera_name}_gazebo_camera_frame">
       <sensor type="depth" name="${camera_name}">
         <update_rate>15.0</update_rate> <!-- Gazebo does not necessarily respect this update rate when publishing the camera data to ros2 -->
         <camera>
-          <horizontal_fov>1.57</horizontal_fov>
+          <horizontal_fov>1.51</horizontal_fov> <!-- Set horizontal FOV to realsense d435i horizontal color FOV (69 degrees)-->
           <!-- There is not a control for vertical FOV, it is set automatically as height / width * horizontal_fov -->
           <image>
-            <width>640</width>
-            <height>389</height>
+            <width>100</width>
+            <height>56</height> <!-- Set pixel height so that vertical FOV matches realsense d435i -->
             <format>R8G8B8</format>
           </image>
           <clip>
+            <!-- Physical realsense cuts off around 10cm, sim camera seems to cutoff at 30cm no matter what. -->
             <near>0.1</near>
             <!--  Be sure to set far clip greater than cropbox node's cutoff distance.

Commit message: Added proper orientation during dropoff, based on row num and which side of worker was approached during pickup

File: antdrone_description/urdf/base.urdf.xacro (robot description, xacro)
@@ -35,5 +35,5 @@
     <mu2>0.0</mu2>
   </gazebo>
-  <link name="attachment_point">
+  <link name="attachment_point_R">
       <inertial>
         <origin xyz="0 0 0" rpy="0 0 0"/>
@@ -48,12 +48,57 @@
       </inertial>
     </link>
-  <joint name="attachment_to_base" type="fixed">
+  <joint name="attachment_point_R_to_base" type="fixed">
     <parent link="base_link"/>
-    <child link="attachment_point"/>
+    <child link="attachment_point_R"/>
+    <origin xyz="0 0 0.6" rpy="0 0 -1.57"/>
+  </joint>
+  <gazebo reference='attachment_point_R_to_base'>
+    <preserveFixedJoint>true</preserveFixedJoint>
+  </gazebo>
+  <link name="attachment_point_L">
+      <inertial>
+        <origin xyz="0 0 0" rpy="0 0 0"/>
+        <mass value="0.01"/> <!-- Small, non-zero mass -->
+        <inertia
+          ixx="0.0001"
+          ixy="0"
+          ixz="0"
+          iyy="0.0001"
+          iyz="0"
+          izz="0.0001" />
+      </inertial>
+    </link>
+  <joint name="attachment_point_L_to_base" type="fixed">
+    <parent link="base_link"/>
+    <child link="attachment_point_L"/>
     <origin xyz="0 0 0.6" rpy="0 0 1.57"/>
   </joint>
-  <gazebo reference='attachment_to_base'>
+  <gazebo reference='attachment_point_L_to_base'>
     <preserveFixedJoint>true</preserveFixedJoint>
   </gazebo>
+  <link name="front_marker">
+    <visual>
+      <origin xyz="0 0 0" rpy="0 0 0"/>
+      <geometry>
+        <box size="0.05 0.05 0.05"/>
+      </geometry>
+    </visual>
+    <inertial>
+      <origin xyz="0 0 0" rpy="0 0 0"/>
+      <mass value="0.01"/> <!-- Small, non-zero mass -->
+      <inertia
+        ixx="0.0001"
+        ixy="0"
+        ixz="0"
+        iyy="0.0001"
+        iyz="0"
+        izz="0.0001" />
+    </inertial>
+  </link>
+  <joint name="front_marker_to_base" type="fixed">
+    <parent link="base_link"/>
+    <child link="front_marker"/>
+    <origin xyz="${base_length / 2 - 0.05} 0 ${base_height}" rpy="0 0 0"/>
+  </joint>
   </xacro:macro>
 </robot>
