Commit message: Found combination of res, pitch, and FOV necessary for a camera to see an apriltag on the underside of the worker during its entire mating procedure

File: antdrone_description/urdf/camera.urdf.xacro (robot description, xacro)
@@ -6,9 +6,10 @@
         <update_rate>15.0</update_rate> <!-- Gazebo does not necessarily respect this update rate when publishing the camera data to ros2 -->
         <camera>
-          <horizontal_fov>1.517</horizontal_fov>
+          <horizontal_fov>1.92</horizontal_fov> <!-- Set horizontal FOV to realsense d435i horizontal color FOV (69 degrees)-->
+          <!-- There is not a control for vertical FOV, it is set automatically as height / width * horizontal_fov -->
           <image>
             <!-- Set width & height to match settings on physical realsense -->
             <width>640</width>
-            <height>480</height>
+            <height>389</height> <!-- Set pixel height so that vertical FOV matches realsense d435i -->
             <format>R8G8B8</format>
           </image>

File: antdrone_description/urdf/mecanum_libplanar.urdf.xacro (robot description, xacro)
@@ -5,9 +5,9 @@
   <xacro:include filename="$(find antdrone_description)/urdf/base.urdf.xacro" />
   <xacro:include filename="$(find antdrone_description)/urdf/camera.urdf.xacro" />
-  <xacro:property name="rs_height" value="${base_height/2 + 0.05}" />
+  <xacro:property name="rs_height" value="${base_height/2 + 0.107}" />
   <xacro:camera drone_name="$(arg drone_name)" camera_pos="front"
                 x="0.410335" y="0" z="${rs_height}"
                 r_rs= "-1.57" p_rs="0" yaw_rs="-1.57"
-                r_cam="0" p_cam="0" yaw_cam="0"/>
+                r_cam="1.57" p_cam="-1.1" yaw_cam="0"/>
   <xacro:camera drone_name="$(arg drone_name)" camera_pos="left"
                 x="0.0" y="0.247" z="${rs_height}"

Commit message: Pre-alignment pickup phase complete

File: antdrone_description/urdf/camera.urdf.xacro (robot description, xacro)
@@ -6,5 +6,5 @@
         <update_rate>15.0</update_rate> <!-- Gazebo does not necessarily respect this update rate when publishing the camera data to ros2 -->
         <camera>
-          <horizontal_fov>1.92</horizontal_fov> <!-- Set horizontal FOV to realsense d435i horizontal color FOV (69 degrees)-->
+          <horizontal_fov>1.57</horizontal_fov> <!-- Set horizontal FOV to realsense d435i horizontal color FOV (69 degrees)-->
           <!-- There is not a control for vertical FOV, it is set automatically as height / width * horizontal_fov -->
           <image>

File: antdrone_description/urdf/mecanum_libplanar.urdf.xacro (robot description, xacro)
@@ -5,9 +5,9 @@
   <xacro:include filename="$(find antdrone_description)/urdf/base.urdf.xacro" />
   <xacro:include filename="$(find antdrone_description)/urdf/camera.urdf.xacro" />
-  <xacro:property name="rs_height" value="${base_height/2 + 0.107}" />
+  <xacro:property name="rs_height" value="${0.37 - base_height/2}" />
   <xacro:camera drone_name="$(arg drone_name)" camera_pos="front"
-                x="0.410335" y="0" z="${rs_height}"
-                r_rs= "-1.57" p_rs="0" yaw_rs="-1.57"
-                r_cam="1.57" p_cam="-1.1" yaw_cam="0"/>
+                x="${base_length/2 - 0.0575}" y="-0.195" z="${rs_height}"
+                r_rs= "-1.57" p_rs="0" yaw_rs="${(60-90)/180*3.14}"
+                r_cam="0" p_cam="0" yaw_cam="${60/180*3.14}"/>
   <xacro:camera drone_name="$(arg drone_name)" camera_pos="left"
                 x="0.0" y="0.247" z="${rs_height}"

Commit message: Updated gz & irl camera positioning so that gazebo cameras are positioned relative to frames that define real cameras. Simplifies transforms quite a bit

File: antdrone_description/urdf/camera.urdf.xacro (robot description, xacro)
@@ -1,5 +1,11 @@
 <?xml version="1.0"?>
+  <!-- The image frame from gazebo does NOT match the output frame of physical cameras -->
+  <!-- Physical cameras have: z out the front, x out the right, y down -->
+  <!-- Gazebo cameras have: x out the front, y out the left, z up -->
+  <!-- Since we need the physical frame for physical & sim robots to match frames,
+        define a transform from the physical to real frame that will put the gazebo
+        camera in the correct position to mimic a real camera -->
 <robot name="antdrone_camera" xmlns:xacro="http://ros.org/wiki/xacro">
-  <xacro:macro name="camera" params="drone_name camera_name x y z r_rs p_rs yaw_rs r_cam p_cam yaw_cam">
+  <xacro:macro name="camera" params="drone_name camera_name x y z roll pitch yaw">
     <gazebo reference="${camera_name}_gazebo_camera_frame">
       <sensor type="depth" name="${camera_name}">
@@ -9,6 +15,6 @@
           <!-- There is not a control for vertical FOV, it is set automatically as height / width * horizontal_fov -->
           <image>
-            <width>640</width>
-            <height>389</height>
+            <width>800</width>
+            <height>600</height>
             <format>R8G8B8</format>
           </image>
@@ -51,5 +57,5 @@
       <origin
         xyz="${x} ${y} ${z}"
-        rpy="${r_rs} ${p_rs} ${yaw_rs}" />
+        rpy="${roll} ${pitch} ${yaw}" />
       <parent link="base_link" />
       <child link="${camera_name}_depth_optical_frame" />
@@ -58,9 +64,9 @@
     </link>
     <joint
-      name="base_link_to_${camera_name}_gazebo_camera_frame" type="fixed">
+      name="${camera_name}_depth_optical_frame_to_${camera_name}_gazebo_camera_frame" type="fixed">
       <origin
-        xyz="${x} ${y} ${z}"
-        rpy="${r_cam} ${p_cam} ${yaw_cam}" />
-      <parent link="base_link" />
+        xyz="0 0 0"
+        rpy="1.57 -1.57 0" />
+      <parent link="${camera_name}_depth_optical_frame" />
       <child link="${camera_name}_gazebo_camera_frame" />
     </joint>

File: antdrone_description/urdf/mecanum_libplanar.urdf.xacro (robot description, xacro)
@@ -6,27 +6,22 @@
   <xacro:include filename="$(find antdrone_description)/urdf/camera.urdf.xacro" />
   <xacro:include filename="$(find antdrone_description)/urdf/rs.urdf.xacro" />
-  <xacro:property name="rs_height" value="${base_height + 0.04}" />
+  <xacro:property name="rs_height" value="${base_height + 0.025}" />
   <xacro:camera drone_name="$(arg drone_name)" camera_name="apriltag_cam"
-                x="${base_length/2 - 0.0575}" y="-0.195" z="0.37"
-                r_rs= "-1.57" p_rs="0" yaw_rs="${(60-90)/180*3.14}"
-                r_cam="0" p_cam="0" yaw_cam="${60/180*3.14}"/>
+                x="0" y="0.215" z="0.19"
+                roll= "${-70/180*3.14}" pitch="0" yaw="-1.57"/>
   <xacro:rs drone_name="$(arg drone_name)" camera_name="front_rs"
                 x="0.41" y="0.0" z="${rs_height}"
-                r_rs= "-1.57" p_rs="0" yaw_rs="-1.57"
-                r_cam="0" p_cam="0" yaw_cam="0"/>
+                roll="-1.57" pitch="0" yaw="-1.57"/>
   <xacro:rs drone_name="$(arg drone_name)" camera_name="left_rs"
                 x="0.0" y="0.247" z="${rs_height}"
-                r_rs="-1.57" p_rs="0.0" yaw_rs="0"
-                r_cam="0" p_cam="0" yaw_cam="1.57"
+                roll="-1.57" pitch="0.0" yaw="0"
   />
   <xacro:rs drone_name="$(arg drone_name)" camera_name="rear_rs"
                 x="-0.41" y="0.0" z="${rs_height}"
-                r_rs="-1.57" p_rs="0" yaw_rs="1.57"
-                r_cam="0" p_cam="0" yaw_cam="3.14"
+                roll="-1.57" pitch="0" yaw="1.57"
   />
   <xacro:rs drone_name="$(arg drone_name)" camera_name="right_rs"
                 x="0" y="-0.247" z="${rs_height}"
-                r_rs="-1.57" p_rs="0" yaw_rs="3.14"
-                r_cam="0" p_cam="0" yaw_cam="-1.57"
+                roll="-1.57" pitch="0" yaw="3.14"
   />
   <gazebo>

File: antdrone_description/urdf/rs.urdf.xacro (robot description, xacro)
@@ -1,5 +1,11 @@
 <?xml version="1.0"?>
+  <!-- The image frame from gazebo does NOT match the output frame of physical cameras -->
+  <!-- Physical cameras have: z out the front, x out the right, y down -->
+  <!-- Gazebo cameras have: x out the front, y out the left, z up -->
+  <!-- Since we need the physical frame for physical & sim robots to match frames,
+        define a transform from the physical to real frame that will put the gazebo
+        camera in the correct position to mimic a real camera -->
 <robot name="antdrone_camera" xmlns:xacro="http://ros.org/wiki/xacro">
-  <xacro:macro name="rs" params="drone_name camera_name x y z r_rs p_rs yaw_rs r_cam p_cam yaw_cam">
+  <xacro:macro name="rs" params="drone_name camera_name x y z roll pitch yaw">
     <gazebo reference="${camera_name}_gazebo_camera_frame">
       <sensor type="depth" name="${camera_name}">
@@ -52,5 +58,5 @@
       <origin
         xyz="${x} ${y} ${z}"
-        rpy="${r_rs} ${p_rs} ${yaw_rs}" />
+        rpy="${roll} ${pitch} ${yaw}" />
       <parent link="base_link" />
       <child link="${camera_name}_depth_optical_frame" />
@@ -59,9 +65,9 @@
     </link>
     <joint
-      name="base_link_to_${camera_name}_gazebo_camera_frame" type="fixed">
+      name="${camera_name}_depth_optical_frame_to_${camera_name}_gazebo_camera_frame" type="fixed">
       <origin
-        xyz="${x} ${y} ${z}"
-        rpy="${r_cam} ${p_cam} ${yaw_cam}" />
-      <parent link="base_link" />
+        xyz="0 0 0"
+        rpy="1.57 -1.57 0" />
+      <parent link="${camera_name}_depth_optical_frame" />
       <child link="${camera_name}_gazebo_camera_frame" />
     </joint>

Commit message: Apriltag cam mounted to robot, spitting out very accurate transforms to physical apriltags on worker

File: antdrone_description/urdf/camera.urdf.xacro (robot description, xacro)
@@ -51,5 +51,5 @@
       </sensor>
     </gazebo>
-    <link name="${camera_name}_depth_optical_frame">
+    <link name="${camera_name}_cam">
     </link>
     <joint
@@ -59,14 +59,14 @@
         rpy="${roll} ${pitch} ${yaw}" />
       <parent link="base_link" />
-      <child link="${camera_name}_depth_optical_frame" />
+      <child link="${camera_name}_cam" />
     </joint>
     <link name="${camera_name}_gazebo_camera_frame">
     </link>
     <joint
-      name="${camera_name}_depth_optical_frame_to_${camera_name}_gazebo_camera_frame" type="fixed">
+      name="${camera_name}_cam_to_${camera_name}_gazebo_camera_frame" type="fixed">
       <origin
         xyz="0 0 0"
         rpy="1.57 -1.57 0" />
-      <parent link="${camera_name}_depth_optical_frame" />
+      <parent link="${camera_name}_cam" />
       <child link="${camera_name}_gazebo_camera_frame" />
     </joint>

File: antdrone_description/urdf/mecanum_libplanar.urdf.xacro (robot description, xacro)
@@ -7,7 +7,7 @@
   <xacro:include filename="$(find antdrone_description)/urdf/rs.urdf.xacro" />
   <xacro:property name="rs_height" value="${base_height + 0.025}" />
-  <xacro:camera drone_name="$(arg drone_name)" camera_name="apriltag_cam"
-                x="0" y="0.215" z="0.19"
-                roll= "${-70/180*3.14}" pitch="0" yaw="-1.57"/>
+  <xacro:camera drone_name="$(arg drone_name)" camera_name="apriltag"
+                x="0" y="0.215" z="0.195"
+                roll= "${-55/180*3.14}" pitch="0" yaw="-1.57"/>
   <xacro:rs drone_name="$(arg drone_name)" camera_name="front_rs"
                 x="0.41" y="0.0" z="${rs_height}"

Commit message: Updated simulated camera naming conventions to match naming convention for physical apriltag cam

File: antdrone_description/urdf/camera.urdf.xacro (robot description, xacro)
@@ -31,5 +31,5 @@
           </noise>
         </camera>
-        <plugin name="${camera_name}_camera_controller" filename="libgazebo_ros_camera.so">
+        <plugin name="${camera_name}_controller" filename="libgazebo_ros_camera.so">
           <ros>
               <namespace>${drone_name}</namespace>
@@ -37,5 +37,5 @@
           <alwaysOn>true</alwaysOn>
           <updateRate>0.0</updateRate>
-          <cameraName>${camera_name}_camera</cameraName>
+          <cameraName>${camera_name}</cameraName>
           <pointsTopicName>points</pointsTopicName>
           <imageTopicName>image_raw</imageTopicName>
@@ -51,5 +51,5 @@
       </sensor>
     </gazebo>
-    <link name="${camera_name}_cam">
+    <link name="${camera_name}">
     </link>
     <joint
@@ -59,14 +59,14 @@
         rpy="${roll} ${pitch} ${yaw}" />
       <parent link="base_link" />
-      <child link="${camera_name}_cam" />
+      <child link="${camera_name}" />
     </joint>
     <link name="${camera_name}_gazebo_camera_frame">
     </link>
     <joint
-      name="${camera_name}_cam_to_${camera_name}_gazebo_camera_frame" type="fixed">
+      name="${camera_name}_to_${camera_name}_gazebo_camera_frame" type="fixed">
       <origin
         xyz="0 0 0"
         rpy="1.57 -1.57 0" />
-      <parent link="${camera_name}_cam" />
+      <parent link="${camera_name}" />
       <child link="${camera_name}_gazebo_camera_frame" />
     </joint>

File: antdrone_description/urdf/mecanum_libplanar.urdf.xacro (robot description, xacro)
@@ -7,5 +7,5 @@
   <xacro:include filename="$(find antdrone_description)/urdf/rs.urdf.xacro" />
   <xacro:property name="rs_height" value="${base_height + 0.025}" />
-  <xacro:camera drone_name="$(arg drone_name)" camera_name="apriltag"
+  <xacro:camera drone_name="$(arg drone_name)" camera_name="apriltag_cam"
                 x="0" y="0.215" z="0.195"
                 roll= "${-55/180*3.14}" pitch="0" yaw="-1.57"/>
